Commit message: Adapting scripts for robot navigation

File: models/lidarbot.urdf (robot description, URDF)
Before this commit: robot lidarbot, 8 links, 7 joints
Joints:
- removed joint caster_wheel_to_base_link
- removed joint left_wheel_hinge
- removed joint right_wheel_hinge
- added joint caster_wheel_joint: type fixed, parent base_link, child caster_wheel, origin xyz=0.0925 0 -0.031 rpy=0 0 1.5707, axis 0 0 1
- added joint left_wheel_joint: type revolute, parent base_link, child left_wheel, origin xyz=-0.028 0.055 -${wheel_zoff} rpy=1.5707 0 3.1414, axis 0 1 0, limit lower=-3.1415 upper=3.1415 effort=30 velocity=5.0
- added joint right_wheel_joint: type revolute, parent base_link, child right_wheel, origin xyz=-0.028 -0.065 -${wheel_zoff} rpy=1.5707 0 -3.1414, axis 0 1 0, limit lower=-3.1415 upper=3.1415 effort=30 velocity=5.0

Commit message: minor changes in lidarbot.urdf

File: models/lidarbot.urdf (robot description, URDF)
Before this commit: robot lidarbot, 8 links, 7 joints
Joints:
- joint left_wheel_joint: axis 0 1 0 -> 0 0 1

Commit message: Axis changes in lidarbot.urdf file

File: models/lidarbot.urdf (robot description, URDF)
Before this commit: robot lidarbot, 8 links, 7 joints
Joints:
- joint right_wheel_joint: axis 0 1 0 -> 0 0 1
