Commit message: Breaking up lidarbot.urdf into xacro files

File: models/lidarbot copy.urdf (robot description, URDF)
Before this commit: robot lidarbot, 8 links, 7 joints
Joints:
- joint left_wheel_joint: limit (none) -> lower=-3.1415 upper=3.1415 effort=30 velocity=5.0; type continuous -> revolute
- joint right_wheel_joint: limit (none) -> lower=-3.1415 upper=3.1415 effort=30 velocity=5.0; type continuous -> revolute

File: models/lidarbot_core.xacro (robot description, xacro)
@@ -1,4 +1,4 @@
 <?xml version="1.0" ?>
-<robot name="lidarbot" xmlns:xacro="http://ros.org/wiki/xacro">
+<robot xmlns:xacro="http://ros.org/wiki/xacro">
   <!-- Robot constants -->
   <!-- Define the size of the robot's main chassis in meters-->
@@ -180,8 +180,9 @@
     <xacro:thick_walled_cylinder_inertia m="0.031" r2="${wheel_outer_radius}" r1="${wheel_inner_radius}" h="${wheel_width}"/>
   </link>
-  <joint name="left_wheel_joint" type="continuous">
+  <joint name="left_wheel_joint" type="revolute">
     <parent link="base_link"/>
     <child link="left_wheel"/>
     <origin xyz="-0.028 0.055 -${wheel_zoff}" rpy="1.5707 0 3.1414"/>
+    <limit upper="3.1415" lower="-3.1415" effort="30" velocity="5.0"/>
     <axis xyz="0 0 1"/>
     <!-- <axis xyz="0 1 0"/> -->
@@ -202,8 +203,9 @@
     <xacro:thick_walled_cylinder_inertia m="0.031" r2="${wheel_outer_radius}" r1="${wheel_inner_radius}" h="${wheel_width}"/>
   </link>
-  <joint name="right_wheel_joint" type="continuous">
+  <joint name="right_wheel_joint" type="revolute">
     <parent link="base_link"/>
     <child link="right_wheel"/>
     <origin xyz="-0.028 -0.065 -${wheel_zoff}" rpy="1.5707 0 -3.1414"/>
+    <limit upper="3.1415" lower="-3.1415" effort="30" velocity="5.0"/>
     <axis xyz="0 0 1"/>
     <!-- <axis xyz="0 1 0"/> -->
