Commit message: Changes to core xacro file

File: models/lidarbot_core copy.xacro (robot description, xacro)
@@ -20,5 +20,5 @@
     <child link="base_link"/>
     <!-- <origin xyz="0 0 0" rpy="0 0 0"/> -->
-    <origin xyz="0 0 ${-(wheel_outer_radius+wheel_zoff)}" rpy="0 0 0"/>
+    <origin xyz="0 0 ${(wheel_outer_radius+wheel_zoff)}" rpy="0 0 0"/>
   </joint>
   <!-- Robot Base -->
