Commit message: removed box inertia added cylinder inertia

File: models/inertial_macros.xacro (robot description, xacro)
@@ -15,6 +15,6 @@
             <xacro:insert_block name="origin"/>
             <mass value="${mass}"/>
-            <inertia ixx="${(mass/12) * (3*(outer_radius*outer_radius + inner_radius*inner_radius) + height*height)}" ixy = "0" ixz = "0"
-                    iyy="${(mass/12) * (3*(outer_radius*outer_radius + inner_radius*inner_radius) + height*height)}" iyz = "0"
+            <inertia ixx="${(mass/12) * (3*(outer_radius*outer_radius + inner_radius*inner_radius) + height*height)}" ixy = "0.0" ixz = "0.0"
+                    iyy="${(mass/12) * (3*(outer_radius*outer_radius + inner_radius*inner_radius) + height*height)}" iyz = "0.0"
                     izz="${(mass/2) * (outer_radius*outer_radius + inner_radius*inner_radius)}"/>
         </inertial>

File: models/lidarbot_core.xacro (robot description, xacro)
@@ -142,7 +142,7 @@
       </geometry>
     </collision>
-      <xacro:box_inertia mass="0.863" width="${base_width}" depth="${base_length}" height="${base_height}">
+      <!-- <xacro:box_inertia mass="0.863" width="${base_width}" depth="${base_length}" height="${base_height}">
         <origin xyz="0 0 -0.0125" rpy="0 0 0"/>
-      </xacro>
+      </xacro> -->
   </link>
   <!-- Left Wheel Link -->
@@ -160,7 +160,7 @@
       </geometry>
     </collision>
-    <!-- <xacro:thick_walled_cylinder_inertia mass="0.031" outer_radius="${wheel_outer_radius}" inner_radius="${wheel_inner_radius}" height="${wheel_height}">
-      <origin xyz="0 0 0" rpy="0 0 0"/>
-    </xacro> -->
+    <xacro:thick_walled_cylinder_inertia mass="0.031" outer_radius="${wheel_outer_radius}" inner_radius="${wheel_inner_radius}" height="${wheel_height}">
+      <origin xyz="0 0 0" rpy="0 0 0"/>
+    </xacro>
   </link>
   <joint name="left_wheel_joint" type="continuous">
@@ -184,7 +184,7 @@
       </geometry>
     </collision>
-    <!-- <xacro:thick_walled_cylinder_inertia mass="0.031" outer_radius="${wheel_outer_radius}" inner_radius="${wheel_inner_radius}" height="${wheel_height}">
-      <origin xyz="0 0 0" rpy="0 0 0"/>
-    </xacro> -->
+    <xacro:thick_walled_cylinder_inertia mass="0.031" outer_radius="${wheel_outer_radius}" inner_radius="${wheel_inner_radius}" height="${wheel_height}">
+      <origin xyz="0 0 0" rpy="0 0 0"/>
+    </xacro>
   </link>
   <joint name="right_wheel_joint" type="continuous">

Commit message: Add inertial tags to sdf file and renamed variables in inertial_macros.xacro

File: models/inertial_macros.xacro (robot description, xacro)
@@ -2,11 +2,15 @@
 <robot xmlns:xacro="http://ros.org/wiki/xacro">
     <!-- Some standard inertial calculations, obtained from: https://en.wikipedia.org/wiki/List_of_moments_of_inertia -->
-    <xacro:macro name="box_inertia" params="mass width height depth *origin">
+    <xacro:macro name="box_inertia" params="mass length width height *origin">
+    <!-- <xacro:macro name="box_inertia" params="mass width height depth *origin"> -->
         <inertial>
             <xacro:insert_block name="origin"/>
             <mass value="${mass}"/>
-            <inertia ixx="${(mass/12) * (height*height + depth*depth)}" ixy="0.0" ixz="0.0"
+            <inertia ixx="${(mass/12) * (width*width + height*height)}" ixy="0.0" ixz="0.0"
+                    iyy="${(mass/12) * (length*length + height*height)}" iyz="0.0"
+                    izz="${(mass/12) * (length*length + width*width)}"/>
+            <!-- <inertia ixx="${(mass/12) * (height*height + depth*depth)}" ixy="0.0" ixz="0.0"
                     iyy="${(mass/12) * (width*width + depth*depth)}" iyz="0.0"
-                    izz="${(mass/12) * (width*width + height*height)}"/>
+                    izz="${(mass/12) * (width*width + height*height)}"/> -->
         </inertial>
     </xacro:macro>

File: models/lidarbot_core.xacro (robot description, xacro)
@@ -140,5 +140,5 @@
       </geometry>
     </collision>
-    <xacro:box_inertia mass="0.864" width="${base_width}" depth="${base_length}" height="${base_height}">
+    <xacro:box_inertia mass="0.864" length="${base_length}" width="${base_width}" height="${base_height}">
       <origin xyz="0 0 -0.0125" rpy="0 0 0"/>
     </xacro:box_inertia>

Commit message: Made adjustments to core xacro file

File: models/inertial_macros.xacro (robot description, xacro)
@@ -3,5 +3,4 @@
     <!-- Some standard inertial calculations, obtained from: https://en.wikipedia.org/wiki/List_of_moments_of_inertia -->
     <xacro:macro name="box_inertia" params="mass length width height *origin">
-    <!-- <xacro:macro name="box_inertia" params="mass width height depth *origin"> -->
         <inertial>
             <xacro:insert_block name="origin"/>
@@ -10,7 +9,4 @@
                     iyy="${(mass/12) * (length*length + height*height)}" iyz="0.0"
                     izz="${(mass/12) * (length*length + width*width)}"/>
-            <!-- <inertia ixx="${(mass/12) * (height*height + depth*depth)}" ixy="0.0" ixz="0.0"
-                    iyy="${(mass/12) * (width*width + depth*depth)}" iyz="0.0"
-                    izz="${(mass/12) * (width*width + height*height)}"/> -->
         </inertial>
     </xacro:macro>
@@ -33,3 +29,12 @@
         </inertial>
     </xacro:macro>
+    <xacro:macro name="cylinder_inertia" params="mass length radius *origin">
+        <inertial>
+            <xacro:insert_block name="origin"/>
+            <mass value="${mass}" />
+            <inertia ixx="${(1/12) * mass * (3*radius*radius + length*length)}" ixy="0.0" ixz="0.0"
+                    iyy="${(1/12) * mass * (3*radius*radius + length*length)}" iyz="0.0"
+                    izz="${(1/2) * mass * (radius*radius)}" />
+        </inertial>
+    </xacro:macro>
 </robot>

File: models/lidarbot_core.xacro (robot description, xacro)
@@ -2,12 +2,13 @@
 <robot xmlns:xacro="http://ros.org/wiki/xacro">
   <xacro:include filename="inertial_macros.xacro"/>
-  <!-- Robot's chassis measurements -->
+  <!-- Robot's chassis properties -->
   <xacro:property name="base_length" value="0.21"/>
   <xacro:property name="base_width" value="0.11"/>
   <xacro:property name="base_height" value="0.035"/>
-  <!-- Robot's wheel measurements -->
+  <!-- Robot's wheel properties -->
   <xacro:property name="wheel_outer_radius" value="0.0325"/>
   <xacro:property name="wheel_inner_radius" value="0.0225"/>
   <xacro:property name="wheel_height" value="0.025"/>
+  <xacro:property name="wheel_mass" value="0.031"/>
   <!-- Distance between centre of wheel and robot base/chassis -->
   <xacro:property name="wheel_zoff" value="0.0125"/>
@@ -153,7 +154,10 @@
       </geometry>
     </collision>
-    <xacro:thick_walled_cylinder_inertia mass="0.031" outer_radius="${wheel_outer_radius}" inner_radius="${wheel_inner_radius}" height="${wheel_height}">
-      <origin xyz="0 0 0" rpy="0 0 0"/>
-    </xacro:thick_walled_cylinder_inertia>
+    <!-- <xacro:thick_walled_cylinder_inertia mass="0.031" outer_radius="${wheel_outer_radius}" inner_radius="${wheel_inner_radius}" height="${wheel_height}">
+      <origin xyz="0 0 0" rpy="0 0 0"/>
+    </xacro:thick_walled_cylinder_inertia> -->
+    <xacro:cylinder_inertia mass="${wheel_mass}" length="${wheel_height}" radius="${wheel_outer_radius}">
+      <origin xyz="0 0 0" rpy="0 0 0"/>
+    </xacro:cylinder_inertia>
   </link>
   <joint name="left_wheel_joint" type="continuous">
@@ -176,7 +180,10 @@
       </geometry>
     </collision>
-    <xacro:thick_walled_cylinder_inertia mass="0.031" outer_radius="${wheel_outer_radius}" inner_radius="${wheel_inner_radius}" height="${wheel_height}">
-      <origin xyz="0 0 0" rpy="0 0 0"/>
-    </xacro:thick_walled_cylinder_inertia>
+    <!-- <xacro:thick_walled_cylinder_inertia mass="0.031" outer_radius="${wheel_outer_radius}" inner_radius="${wheel_inner_radius}" height="${wheel_height}">
+      <origin xyz="0 0 0" rpy="0 0 0"/>
+    </xacro:thick_walled_cylinder_inertia> -->
+    <xacro:cylinder_inertia mass="${wheel_mass}" length="${wheel_height}" radius="${wheel_outer_radius}">
+      <origin xyz="0 0 0" rpy="0 0 0"/>
+    </xacro:cylinder_inertia>
   </link>
   <joint name="right_wheel_joint" type="continuous">
@@ -190,6 +197,5 @@
     <visual>
       <geometry>
-        <mesh filename="package://models/lidarbot_description/meshes/caster_wheel.dae"/>
-        <!-- <mesh filename="package://real_lidarbot/models/lidarbot_description/meshes/caster_wheel.dae"/> -->
+        <mesh filename="package://real_lidarbot/models/lidarbot_description/meshes/caster_wheel.dae"/>
       </geometry>
     </visual>
