Commit message: Changes to xacro file

File: models/depth_camera.xacro (robot description, xacro)
@@ -18,6 +18,6 @@
     <parent link="base_link"/>
     <child link="camera_link"/>
-    <origin xyz="0.1 0 0.0425" rpy="1.5707 0 1.5707"/>
+    <origin xyz="0.1 0 0.0425" rpy="${pi/2} 0 {pi/2}"/>
   </joint>
-  <!-- Need to add more details for the camera  -->
+  <!-- Need to add more details for the camera also in sdf file -->
 </robot>

File: models/imu.xacro (robot description, xacro)
@@ -12,5 +12,5 @@
     <parent link="base_link"/>
     <child link="imu_link"/>
-    <origin xyz="-0.06 0 0.0175" rpy="0 0 3.1414"/>
+    <origin xyz="-0.06 0 0.0175" rpy="0 0 ${pi}"/>
   </joint>
 </robot>

File: models/inertial_macros.xacro (robot description, xacro)
@@ -1,5 +1,5 @@
 <?xml version="1.0" ?>
 <robot xmlns:xacro="http://ros.org/wiki/xacro">
-    <!-- Specify some standard inertial calculations https://en.wikipedia.org/wiki/List_of_moments_of_inertia -->
+    <!-- Some standard inertial calculations, obtained from: https://en.wikipedia.org/wiki/List_of_moments_of_inertia -->
     <xacro:macro name="box_inertia" params="mass width height depth *origin">
         <inertial>

File: models/lidarbot_core.xacro (robot description, xacro)
@@ -3,14 +3,13 @@
   <xacro:include filename="inertial_macros.xacro"/>
   <!-- Robot constants (measurements in metres) -->
-  <!-- Define the size of the robot's main chassis in meters-->
+  <!-- Robot's chassis measurements -->
   <xacro:property name="base_length" value="0.21"/>
   <xacro:property name="base_width" value="0.11"/>
   <xacro:property name="base_height" value="0.035"/>
-  <!-- Define the shape of the robot's two back wheels in metres-->
+  <!-- Robot's wheel measurements -->
   <xacro:property name="wheel_outer_radius" value="0.0325"/>
   <xacro:property name="wheel_inner_radius" value="0.0225"/>
   <xacro:property name="wheel_height" value="0.025"/>
-  <!-- x-axis points forward, y-axis points to left, z-axis points upwards -->
-  <!-- Define the gap between the wheel and chassis along y-axis in meters -->
+  <!-- Gap between the wheel and chassis along y-axis -->
   <xacro:property name="wheel_ygap" value="0.003"/>
   <!-- Distance between centre of wheel and robot base/chassis -->
@@ -52,5 +51,5 @@
      <!-- Rpi stand -->
      <visual name="rpi_4_stand_visual">
-      <origin xyz="-0.06 0.015 0.031" rpy="3.1414 0 -3.1414"/>
+      <origin xyz="-0.06 0.015 0.031" rpy="${pi} 0 ${-pi}"/>
         <geometry>
             <mesh filename="package://real_lidarbot/models/lidarbot_description/meshes/rpi_stand.dae" />
@@ -58,5 +57,5 @@
     </visual>
     <collision name="rpi_4_stand_collision">
-      <origin xyz="-0.06 0 0.017" rpy="0 0 1.5707"/>
+      <origin xyz="-0.06 0 0.017" rpy="0 0 ${pi/2}"/>
       <geometry>
         <box size="0.098 0.065 0.034"/>
@@ -65,5 +64,5 @@
     <!-- Raspberry Pi -->
     <visual name="rpi_4_visual">
-      <origin xyz="-0.059 0.00245 0.033" rpy="0 0 1.5707"/>
+      <origin xyz="-0.059 0.00245 0.033" rpy="0 0 ${pi/2}"/>
       <geometry>
         <mesh filename="package://real_lidarbot/models/lidarbot_description/meshes/rpi_4.dae"/>
@@ -71,5 +70,5 @@
     </visual>
     <collision name="rpi_4_collision">
-      <origin xyz="-0.058 0.005 0.041" rpy="0 0 1.5707"/>
+      <origin xyz="-0.058 0.005 0.041" rpy="0 0 ${pi/2}"/>
       <geometry>
         <box size="0.09 0.06 0.02"/>
@@ -78,5 +77,5 @@
     <!-- Power bank stand -->
     <visual name="power_bank_stand_visual">
-      <origin xyz="0.033 0.015 0.031" rpy="3.1414 0 3.1414"/>
+      <origin xyz="0.033 0.015 0.031" rpy="${pi} 0 ${pi}"/>
       <geometry>
         <mesh filename="package://real_lidarbot/models/lidarbot_description/meshes/power_bank_stand.dae"/>
@@ -84,5 +83,5 @@
     </visual>
     <collision name="power_bank_stand_collision">
-      <origin xyz="0.033 0 0.0085" rpy="0 0 1.5707"/>
+      <origin xyz="0.033 0 0.0085" rpy="0 0 ${pi/2}"/>
       <geometry>
         <box size="0.098 0.065 0.015"/>
@@ -91,5 +90,5 @@
     <!-- Power bank -->
     <visual name="power_bank_visual">
-      <origin xyz="0.0635 0.04775 0.015" rpy="0 0 1.5707"/>
+      <origin xyz="0.0635 0.04775 0.015" rpy="0 0 ${pi/2}"/>
       <geometry>
         <mesh filename="package://real_lidarbot/models/lidarbot_description/meshes/power_bank.dae"/>
@@ -97,5 +96,5 @@
     </visual>
     <collision name="power_bank_collision">
-      <origin xyz="0.033 0 0.025" rpy="0 0 1.5707"/>
+      <origin xyz="0.033 0 0.025" rpy="0 0 ${pi/2}"/>
       <geometry>
         <box size="0.096 0.062 0.02"/>
@@ -104,5 +103,5 @@
     <!-- Rplidar stand -->
     <visual name="rplidar_stand_visual">
-      <origin xyz="0.033 0.015 0.017" rpy="0 0 -6.2828"/>
+      <origin xyz="0.033 0.015 0.017" rpy="0 0 ${-2*pi}"/>
       <geometry>
         <mesh filename="package://real_lidarbot/models/lidarbot_description/meshes/rplidar_stand.dae"/>
@@ -110,5 +109,5 @@
     </visual>
     <collision name="rplidar_stand_collision">
-      <origin xyz="0.033 0 0.04" rpy="0 0 1.5707"/>
+      <origin xyz="0.033 0 0.04" rpy="0 0 ${pi/2}"/>
       <geometry>
         <box size="0.098 0.065 0.015"/>
@@ -117,5 +116,5 @@
     <!-- Rplidar base -->
     <visual name="rplidar_base_visual">
-      <origin xyz="0.03485 0.0087 0.037" rpy="0 0 -1.5707"/>
+      <origin xyz="0.03485 0.0087 0.037" rpy="0 0 ${-pi/2}"/>
         <geometry>
           <mesh filename="package://real_lidarbot/models/lidarbot_description/meshes/rplidar_base.dae"/>
@@ -123,5 +122,5 @@
       </visual>
     <collision name="rplidar_base_collision">
-      <origin xyz="0.033 0 0.056" rpy="0 0 -1.5707"/>
+      <origin xyz="0.033 0 0.056" rpy="0 0 ${-pi/2}"/>
       <geometry>
         <box size="0.12 0.072 0.035"/>
@@ -141,5 +140,5 @@
       </geometry>
     </collision>
-    <xacro:box_inertia mass="0.863" width="${base_width}" depth="${base_length}" height="${base_height}">
+    <xacro:box_inertia mass="0.864" width="${base_width}" depth="${base_length}" height="${base_height}">
       <origin xyz="0 0 -0.0125" rpy="0 0 0"/>
     </xacro:box_inertia>
@@ -159,5 +158,5 @@
       </geometry>
     </collision>
-    <xacro:thick_walled_cylinder_inertia mass="0.031" outer_radius="${wheel_outer_radius}" inner_radius="${wheel_inner_radius}" height="${wheel_height}">
+    <xacro:thick_walled_cylinder_inertia mass="0.03" outer_radius="${wheel_outer_radius}" inner_radius="${wheel_inner_radius}" height="${wheel_height}">
       <origin xyz="0 0 0" rpy="0 0 0"/>
     </xacro:thick_walled_cylinder_inertia>
@@ -166,5 +165,5 @@
     <parent link="base_link"/>
     <child link="left_wheel"/>
-    <origin xyz="-0.028 0.055 -${wheel_zoff}" rpy="1.5707 0 3.1414"/>
+    <origin xyz="-0.028 0.055 -${wheel_zoff}" rpy="${pi/2} 0 ${pi}"/>
     <axis xyz="0 0 1"/>
   </joint>
@@ -183,5 +182,5 @@
       </geometry>
     </collision>
-    <xacro:thick_walled_cylinder_inertia mass="0.031" outer_radius="${wheel_outer_radius}" inner_radius="${wheel_inner_radius}" height="${wheel_height}">
+    <xacro:thick_walled_cylinder_inertia mass="0.03" outer_radius="${wheel_outer_radius}" inner_radius="${wheel_inner_radius}" height="${wheel_height}">
       <origin xyz="0 0 0" rpy="0 0 0"/>
     </xacro:thick_walled_cylinder_inertia>
@@ -190,5 +189,5 @@
     <parent link="base_link"/>
     <child link="right_wheel"/>
-    <origin xyz="-0.028 -0.065 -${wheel_zoff}" rpy="1.5707 0 -3.1414"/>
+    <origin xyz="-0.028 -0.065 -${wheel_zoff}" rpy="${pi/2} 0 ${-pi}"/>
     <axis xyz="0 0 1"/>
   </joint>
@@ -201,5 +200,5 @@
     </visual>
     <collision>
-      <origin xyz="0 0 -0.001" rpy="0 0 1.5707"/>
+      <origin xyz="0 0 -0.001" rpy="0 0 ${pi/2}"/>
       <geometry>
         <sphere radius="0.015"/>
@@ -213,5 +212,5 @@
     <parent link="base_link"/>
     <child link="caster_wheel"/>
-    <origin xyz="0.0925 0 -0.031" rpy="0 0 1.5707"/>
+    <origin xyz="0.0925 0 -0.031" rpy="0 0 ${pi/2}"/>
     <axis xyz="0 0 1"/>
   </joint>

Commit message: Minor correction in depth_camera.xacro file

File: models/depth_camera.xacro (robot description, xacro)
@@ -18,5 +18,5 @@
     <parent link="base_link"/>
     <child link="camera_link"/>
-    <origin xyz="0.1 0 0.0425" rpy="${pi/2} 0 {pi/2}"/>
+    <origin xyz="0.1 0 0.0425" rpy="${pi/2} 0 ${pi/2}"/>
   </joint>
   <!-- Need to add more details for the camera also in sdf file -->

Commit message: Testing out lidarbot sim in gazebo and rviz

File: models/depth_camera.xacro (robot description, xacro)
@@ -20,4 +20,9 @@
     <origin xyz="0.1 0 0.0425" rpy="${pi/2} 0 ${pi/2}"/>
   </joint>
-  <!-- Need to add more details for the camera also in sdf file -->
+  <link name="camera_link_optical"></link>
+  <joint name="camera_optical_joint" type="fixed">
+    <parent link="camera_link"/>
+    <child link="camera_link_optical"/>
+    <origin xyz="0 0 0" rpy="${-pi/2} 0 ${-pi/2}"/>
+  </joint>
 </robot>

File: models/lidar.xacro (robot description, xacro)
@@ -15,8 +15,8 @@
         </link>
         <joint name="lidar_joint" type="fixed">
-        <parent link="base_link"/>
-        <child link="lidar_link"/>
-        <origin xyz="0.0335 0.0095 0.069" rpy="0 0 0"/>
-        <axis xyz="0 0 1"/>
+            <parent link="base_link"/>
+            <child link="lidar_link"/>
+            <origin xyz="0.0335 0.0095 0.069" rpy="0 0 0"/>
+            <axis xyz="0 0 1"/>
         </joint>
 </robot>

File: models/lidarbot_core.xacro (robot description, xacro)
@@ -158,5 +158,5 @@
       </geometry>
     </collision>
-    <xacro:thick_walled_cylinder_inertia mass="0.03" outer_radius="${wheel_outer_radius}" inner_radius="${wheel_inner_radius}" height="${wheel_height}">
+    <xacro:thick_walled_cylinder_inertia mass="0.031" outer_radius="${wheel_outer_radius}" inner_radius="${wheel_inner_radius}" height="${wheel_height}">
       <origin xyz="0 0 0" rpy="0 0 0"/>
     </xacro:thick_walled_cylinder_inertia>
@@ -182,5 +182,5 @@
       </geometry>
     </collision>
-    <xacro:thick_walled_cylinder_inertia mass="0.03" outer_radius="${wheel_outer_radius}" inner_radius="${wheel_inner_radius}" height="${wheel_height}">
+    <xacro:thick_walled_cylinder_inertia mass="0.031" outer_radius="${wheel_outer_radius}" inner_radius="${wheel_inner_radius}" height="${wheel_height}">
       <origin xyz="0 0 0" rpy="0 0 0"/>
     </xacro:thick_walled_cylinder_inertia>

Commit message: Tweaks to depth camera xacro

File: models/depth_camera.xacro (robot description, xacro)
@@ -18,5 +18,6 @@
     <parent link="base_link"/>
     <child link="camera_link"/>
-    <origin xyz="0.1 0 0.0425" rpy="${pi/2} 0 ${pi/2}"/>
+    <origin xyz="0.1 0 0.0425" rpy="0 0 0"/>
+    <!-- <origin xyz="0.1 0 0.0425" rpy="${pi/2} 0 ${pi/2}"/> -->
   </joint>
   <link name="camera_link_optical"></link>

File: models/inertial_macros.xacro (robot description, xacro)
@@ -9,13 +9,4 @@
                     iyy="${(mass/12) * (length*length + height*height)}" iyz="0.0"
                     izz="${(mass/12) * (length*length + width*width)}"/>
-        </inertial>
-    </xacro:macro>
-    <xacro:macro name="thick_walled_cylinder_inertia" params="mass outer_radius inner_radius height *origin">
-        <inertial>
-            <xacro:insert_block name="origin"/>
-            <mass value="${mass}"/>
-            <inertia ixx="${(mass/12) * (3*(outer_radius*outer_radius + inner_radius*inner_radius) + height*height)}" ixy = "0.0" ixz = "0.0"
-                    iyy="${(mass/12) * (3*(outer_radius*outer_radius + inner_radius*inner_radius) + height*height)}" iyz = "0.0"
-                    izz="${(mass/2) * (outer_radius*outer_radius + inner_radius*inner_radius)}"/>
         </inertial>
     </xacro:macro>

File: models/lidarbot_core.xacro (robot description, xacro)
@@ -154,7 +154,4 @@
       </geometry>
     </collision>
-    <!-- <xacro:thick_walled_cylinder_inertia mass="0.031" outer_radius="${wheel_outer_radius}" inner_radius="${wheel_inner_radius}" height="${wheel_height}">
-      <origin xyz="0 0 0" rpy="0 0 0"/>
-    </xacro:thick_walled_cylinder_inertia> -->
     <xacro:cylinder_inertia mass="${wheel_mass}" length="${wheel_height}" radius="${wheel_outer_radius}">
       <origin xyz="0 0 0" rpy="0 0 0"/>
@@ -181,12 +178,8 @@
       </geometry>
     </collision>
-    <!-- <xacro:thick_walled_cylinder_inertia mass="0.031" outer_radius="${wheel_outer_radius}" inner_radius="${wheel_inner_radius}" height="${wheel_height}">
-      <origin xyz="0 0 0" rpy="0 0 0"/>
-    </xacro:thick_walled_cylinder_inertia> -->
     <xacro:cylinder_inertia mass="${wheel_mass}" length="${wheel_height}" radius="${wheel_outer_radius}">
       <origin xyz="0 0 0" rpy="0 0 0"/>
     </xacro:cylinder_inertia>
   </link>
-  <!-- Stopped here -->
   <joint name="right_wheel_joint" type="revolute">
     <parent link="base_link"/>

Commit message: Tweaks to depth camera xacro

File: models/depth_camera.xacro (robot description, xacro)
@@ -18,6 +18,5 @@
     <parent link="base_link"/>
     <child link="camera_link"/>
-    <origin xyz="0.1 0 0.0425" rpy="0 0 0"/>
-    <!-- <origin xyz="0.1 0 0.0425" rpy="${pi/2} 0 ${pi/2}"/> -->
+    <origin xyz="0.1 0 0.0425" rpy="${pi/2} 0 ${pi/2}"/>
   </joint>
   <link name="camera_link_optical"></link>
