Commit message: Changed how mesh files are included in xacro files

File: models/camera.xacro (robot description, xacro)
@@ -5,5 +5,5 @@
     <visual>
       <geometry>
-        <mesh filename="package://real_lidarbot/models/lidarbot_description/meshes/d415.dae"/>
+        <mesh filename="file://$(find real_lidarbot)/models/lidarbot_description/meshes/d415.dae"/>
       </geometry>
     </visual>

File: models/imu.xacro (robot description, xacro)
@@ -5,5 +5,5 @@
     <visual name="imu_visual">
       <geometry>
-        <mesh filename="package://real_lidarbot/models/lidarbot_description/meshes/MPU6050.dae"/>
+        <mesh filename="file://$(find real_lidarbot)/models/lidarbot_description/meshes/MPU6050.dae"/>
       </geometry>
     </visual>

File: models/lidar.xacro (robot description, xacro)
@@ -4,5 +4,5 @@
         <visual>
             <geometry>
-            <mesh filename="package://real_lidarbot/models/lidarbot_description/meshes/rplidar_top.dae"/>
+            <mesh filename="file://$(find real_lidarbot)/models/lidarbot_description/meshes/rplidar_top.dae"/>
             </geometry>
         </visual>

File: models/lidarbot_core.xacro (robot description, xacro)
@@ -26,5 +26,4 @@
           <geometry>
               <mesh filename="file://$(find real_lidarbot)/models/lidarbot_description/meshes/robot_base.dae" />
-              <!-- <mesh filename="package://real_lidarbot/models/lidarbot_description/meshes/robot_base.dae" /> -->
           </geometry>
       </visual>
@@ -38,5 +37,5 @@
           <origin xyz="0.086 0 -0.0475" rpy="0 0 0"/>
         <geometry>
-          <mesh filename="package://real_lidarbot/models/lidarbot_description/meshes/caster_mount.dae" />
+          <mesh filename="file://$(find real_lidarbot)/models/lidarbot_description/meshes/caster_mount.dae" />
         </geometry>
       </visual>
@@ -51,5 +50,5 @@
         <origin xyz="-0.06 0.015 0.031" rpy="${pi} 0 ${-pi}"/>
           <geometry>
-              <mesh filename="package://real_lidarbot/models/lidarbot_description/meshes/rpi_stand.dae" />
+              <mesh filename="file://$(find real_lidarbot)/models/lidarbot_description/meshes/rpi_stand.dae" />
           </geometry>
       </visual>
@@ -64,5 +63,5 @@
         <origin xyz="-0.059 0.00245 0.033" rpy="0 0 ${pi/2}"/>
         <geometry>
-          <mesh filename="package://real_lidarbot/models/lidarbot_description/meshes/rpi_4.dae"/>
+          <mesh filename="file://$(find real_lidarbot)/models/lidarbot_description/meshes/rpi_4.dae"/>
         </geometry>
       </visual>
@@ -77,5 +76,5 @@
         <origin xyz="0.033 0.015 0.031" rpy="${pi} 0 ${pi}"/>
         <geometry>
-          <mesh filename="package://real_lidarbot/models/lidarbot_description/meshes/power_bank_stand.dae"/>
+          <mesh filename="file://$(find real_lidarbot)/models/lidarbot_description/meshes/power_bank_stand.dae"/>
         </geometry>
       </visual>
@@ -90,5 +89,5 @@
         <origin xyz="0.0635 0.04775 0.015" rpy="0 0 ${pi/2}"/>
         <geometry>
-          <mesh filename="package://real_lidarbot/models/lidarbot_description/meshes/power_bank.dae"/>
+          <mesh filename="file://$(find real_lidarbot)/models/lidarbot_description/meshes/power_bank.dae"/>
         </geometry>
       </visual>
@@ -103,5 +102,5 @@
         <origin xyz="0.033 0.015 0.017" rpy="0 0 ${-2*pi}"/>
         <geometry>
-          <mesh filename="package://real_lidarbot/models/lidarbot_description/meshes/rplidar_stand.dae"/>
+          <mesh filename="file://$(find real_lidarbot)/models/lidarbot_description/meshes/rplidar_stand.dae"/>
         </geometry>
       </visual>
@@ -116,5 +115,5 @@
         <origin xyz="0.03485 0.0087 0.037" rpy="0 0 ${-pi/2}"/>
           <geometry>
-            <mesh filename="package://real_lidarbot/models/lidarbot_description/meshes/rplidar_base.dae"/>
+            <mesh filename="file://$(find real_lidarbot)/models/lidarbot_description/meshes/rplidar_base.dae"/>
           </geometry>
         </visual>
@@ -146,5 +145,5 @@
     <visual>
         <geometry>
-          <mesh filename="package://real_lidarbot/models/lidarbot_description/meshes/left_wheel.dae" />
+          <mesh filename="file://$(find real_lidarbot)/models/lidarbot_description/meshes/left_wheel.dae" />
         </geometry>
     </visual>
@@ -170,5 +169,5 @@
     <visual>
       <geometry>
-        <mesh filename="package://real_lidarbot/models/lidarbot_description/meshes/right_wheel.dae"/>
+        <mesh filename="file://$(find real_lidarbot)/models/lidarbot_description/meshes/right_wheel.dae"/>
       </geometry>
     </visual>
@@ -194,5 +193,5 @@
     <visual>
       <geometry>
-        <mesh filename="package://real_lidarbot/models/lidarbot_description/meshes/caster_wheel.dae"/>
+        <mesh filename="file://$(find real_lidarbot)/models/lidarbot_description/meshes/caster_wheel.dae"/>
       </geometry>
     </visual>

Commit message: Changed camera optical joint origin

File: models/camera.xacro (robot description, xacro)
@@ -24,5 +24,6 @@
     <parent link="camera_link"/>
     <child link="camera_link_optical"/>
-    <origin xyz="0 0 0" rpy="${-pi/2} 0 ${-pi/2}"/>
+    <origin xyz="0 0 0" rpy="${pi/2} 0 ${-pi/2}"/>
+    <!-- <origin xyz="0 0 0" rpy="${-pi/2} 0 ${-pi/2}"/> -->
   </joint>
   <gazebo reference="camera_link">

Commit message: Changed camera optical joint origin

File: models/camera.xacro (robot description, xacro)
@@ -24,5 +24,5 @@
     <parent link="camera_link"/>
     <child link="camera_link_optical"/>
-    <origin xyz="0 0 0" rpy="${pi/2} 0 ${-pi/2}"/>
+    <origin xyz="0 0 0" rpy="0 0 ${-pi/2}"/>
     <!-- <origin xyz="0 0 0" rpy="${-pi/2} 0 ${-pi/2}"/> -->
   </joint>

Commit message: Changed camera optical joint origin

File: models/camera.xacro (robot description, xacro)
@@ -4,4 +4,5 @@
   <link name="camera_link">
     <visual>
+      <origin xyz="0 0 0" rpy="${pi/2} 0 ${pi/2}"
       <geometry>
         <mesh filename="file://$(find real_lidarbot)/models/lidarbot_description/meshes/d415.dae"/>
@@ -24,6 +25,5 @@
     <parent link="camera_link"/>
     <child link="camera_link_optical"/>
-    <origin xyz="0 0 0" rpy="0 0 ${-pi/2}"/>
-    <!-- <origin xyz="0 0 0" rpy="${-pi/2} 0 ${-pi/2}"/> -->
+    <origin xyz="0 0 0" rpy="${-pi/2} 0 ${-pi/2}"/>
   </joint>
   <gazebo reference="camera_link">

Commit message: Changed camera optical joint origin

File: models/camera.xacro (robot description, xacro)
@@ -4,5 +4,5 @@
   <link name="camera_link">
     <visual>
-      <origin xyz="0 0 0" rpy="${pi/2} 0 ${pi/2}"
+      <origin xyz="0 0 0" rpy="${pi/2} 0 ${pi/2}">
       <geometry>
         <mesh filename="file://$(find real_lidarbot)/models/lidarbot_description/meshes/d415.dae"/>

Commit message: Changed camera optical joint origin

File: models/camera.xacro (robot description, xacro)
@@ -4,5 +4,5 @@
   <link name="camera_link">
     <visual>
-      <origin xyz="0 0 0" rpy="${pi/2} 0 ${pi/2}">
+      <origin xyz="0 0 0" rpy="${pi/2} 0 ${pi/2}"/>
       <geometry>
         <mesh filename="file://$(find real_lidarbot)/models/lidarbot_description/meshes/d415.dae"/>

Commit message: Changed camera optical joint origin

File: models/camera.xacro (robot description, xacro)
@@ -4,5 +4,5 @@
   <link name="camera_link">
     <visual>
-      <origin xyz="0 0 0" rpy="${pi/2} 0 ${pi/2}"/>
+      <!-- <origin xyz="0 0 0" rpy="${pi/2} 0 ${pi/2}"/> -->
       <geometry>
         <mesh filename="file://$(find real_lidarbot)/models/lidarbot_description/meshes/d415.dae"/>
@@ -19,5 +19,6 @@
     <parent link="base_link"/>
     <child link="camera_link"/>
-    <origin xyz="0.1 0 0.0425" rpy="${pi/2} 0 ${pi/2}"/>
+    <origin xyz="0.1 0 0.0425" rpy="0 0 0"/>
+    <!-- <origin xyz="0.1 0 0.0425" rpy="${pi/2} 0 ${pi/2}"/> -->
   </joint>
   <link name="camera_link_optical"></link>

Commit message: Changed camera optical joint origin

File: models/camera.xacro (robot description, xacro)
@@ -4,5 +4,5 @@
   <link name="camera_link">
     <visual>
-      <!-- <origin xyz="0 0 0" rpy="${pi/2} 0 ${pi/2}"/> -->
+      <origin xyz="0 0 0" rpy="${-pi/2} 0 ${pi/2}"/>
       <geometry>
         <mesh filename="file://$(find real_lidarbot)/models/lidarbot_description/meshes/d415.dae"/>

Commit message: Changed camera optical joint origin

File: models/camera.xacro (robot description, xacro)
@@ -4,5 +4,5 @@
   <link name="camera_link">
     <visual>
-      <origin xyz="0 0 0" rpy="${-pi/2} 0 ${pi/2}"/>
+      <origin xyz="0 0 0" rpy="${pi/2} 0 ${pi/2}"/>
       <geometry>
         <mesh filename="file://$(find real_lidarbot)/models/lidarbot_description/meshes/d415.dae"/>

Commit message: Commented out gazebo control xacro file for ros2_control xacro

File: models/camera.xacro (robot description, xacro)
@@ -20,5 +20,4 @@
     <child link="camera_link"/>
     <origin xyz="0.1 0 0.0425" rpy="0 0 0"/>
-    <!-- <origin xyz="0.1 0 0.0425" rpy="${pi/2} 0 ${pi/2}"/> -->
   </joint>
   <link name="camera_link_optical"></link>
