Commit message: Added sensor tags for lidar xacro file

File: models/lidar.xacro (robot description, xacro)
@@ -20,3 +20,41 @@
             <axis xyz="0 0 1"/>
         </joint>
+        <xacro:cylinder_inertia mass="${wheel_mass}" length="0.021" radius="0.037">
+            <origin xyz="0 0 0" rpy="0 0 0"/>
+        </xacro:cylinder_inertia>
+        <gazebo reference="lidar_link">
+            <sensor name="lidar" type="ray">
+                <pose> 0 0 0 0 0 0 </pose>
+                <visualize>false</visualize>
+                <update_rate>5.5</update_rate>
+                <ray>
+                    <scan>
+                        <horizontal>
+                            <samples>360</samples>
+                            <resolution>1</resolution>
+                            <min_angle>-3.14</min_angle>
+                            <max_angle>3.14</max_angle>
+                        </horizontal>
+                    </scan>
+                    <range>
+                        <min>0.15</min>
+                        <max>12</max>
+                        <resolution>0.2</resolution>
+                    <noise>
+                        <type>gaussian</type>
+                        <mean>0.0</mean>
+                        <stddev>0.01</stddev>
+                    </noise>
+                    </range>
+                </ray>
+                <plugin name="lidar_controller" filename="libgazebo_ros_ray_sensor.so">
+                    <ros>
+                        <remapping>~/out:=scan</remapping>
+                        <!-- <argument>~/out:=scan</argument> -->
+                    </ros>
+                    <output_type>sensor_msgs/LaserScan</output_type>
+                    <frame_name>lidar_link</frame_name>
+                </plugin>
+            </sensor>
+        </gazebo>
 </robot>
