Commit message: Testing out new urdf file

File: models/lidarbot_core.xacro (robot description, xacro)
@@ -1,4 +1,5 @@
 <?xml version="1.0" ?>
 <robot xmlns:xacro="http://ros.org/wiki/xacro">
+  <xacro:include filename="inertial_macros.xacro"/>
   <!-- Robot constants -->
   <!-- Define the size of the robot's main chassis in meters-->
@@ -15,25 +16,4 @@
   <!-- Distance between centre of wheel and robot base/chassis -->
   <xacro:property name="wheel_zoff" value="0.0125"/>
-  <!-- Inertial xacro macros -->
-  <xacro:macro name="box_inertia" params="m w h d">
-    <inertial>
-      <origin xyz="0 0 0" rpy="0 0 0"/>
-      <mass value="${m}"/>
-      <inertia ixx="${(m/12) * (h*h + d*d)}" ixy="0.0" ixz="0.0" iyy="${(m/12) * (w*w + d*d)}" iyz="0.0" izz="${(m/12) * (w*w + h*h)}"/>
-    </inertial>
-  </xacro:macro>
-  <xacro:macro name="thick_walled_cylinder_inertia" params="m r2 r1 h">
-    <inertial>
-      <origin xyz="0 0 0" rpy="0 0 0" />
-      <mass value="${m}"/>
-      <inertia ixx="${(m/12) * (3*(r2*r2 + r1*r1) + h*h)}" ixy = "0" ixz = "0" iyy="${(m/12) * (3*(r2*r2 + r1*r1) + h*h)}" iyz = "0" izz="${(m/2) * (r2*r2 + r1*r1)}"/>
-    </inertial>
-  </xacro:macro>
-  <xacro:macro name="sphere_inertia" params="m r">
-    <inertial>
-      <mass value="${m}"/>
-      <inertia ixx="${(2/5) * m * (r*r)}" ixy="0.0" ixz="0.0" iyy="${(2/5) * m * (r*r)}" iyz="0.0" izz="${(2/5) * m * (r*r)}"/>
-    </inertial>
-  </xacro:macro>
   <!-- Robot Base Footprint -->
   <!-- Defines the centre of the main robot chassis projected on the ground -->
@@ -162,7 +142,9 @@
       </geometry>
     </collision>
-      <xacro:box_inertia m="0.863" w="${base_width}" d="${base_length}" h="${base_height}"/>
-  </link>
-  <!-- Drive Wheels -->
+      <xacro:box_inertia mass="0.863" width="${base_width}" depth="${base_length}" height="${base_height}">
+        <origin xyz="0 0 -0.0125" rpy="0 0 0"/>
+      </xacro>
+  </link>
+  <!-- Left Wheel Link -->
   <link name="left_wheel">
     <visual>
@@ -178,14 +160,15 @@
       </geometry>
     </collision>
-    <xacro:thick_walled_cylinder_inertia m="0.031" r2="${wheel_outer_radius}" r1="${wheel_inner_radius}" h="${wheel_width}"/>
-  </link>
-  <joint name="left_wheel_joint" type="revolute">
+    <xacro:thick_walled_cylinder_inertia m="0.031" outer_radius="${wheel_outer_radius}" inner_radius="${wheel_inner_radius}" h="${wheel_width}">
+      <origin xyz="0 0 0" rpy="0 0 0"/>
+    </xacro>
+  </link>
+  <joint name="left_wheel_joint" type="continuous">
     <parent link="base_link"/>
     <child link="left_wheel"/>
     <origin xyz="-0.028 0.055 -${wheel_zoff}" rpy="1.5707 0 3.1414"/>
-    <limit upper="3.1415" lower="-3.1415" effort="30" velocity="5.0"/>
     <axis xyz="0 0 1"/>
-    <!-- <axis xyz="0 1 0"/> -->
-  </joint>
+  </joint>
+  <!-- Right Wheel Link -->
   <link name="right_wheel">
     <visual>
@@ -201,13 +184,13 @@
       </geometry>
     </collision>
-    <xacro:thick_walled_cylinder_inertia m="0.031" r2="${wheel_outer_radius}" r1="${wheel_inner_radius}" h="${wheel_width}"/>
-  </link>
-  <joint name="right_wheel_joint" type="revolute">
+    <xacro:thick_walled_cylinder_inertia m="0.031" outer_radius="${wheel_outer_radius}" inner_radius="${wheel_inner_radius}" h="${wheel_width}">
+      <origin xyz="0 0 0" rpy="0 0 0"/>
+    </xacro>
+  </link>
+  <joint name="right_wheel_joint" type="continuous">
     <parent link="base_link"/>
     <child link="right_wheel"/>
     <origin xyz="-0.028 -0.065 -${wheel_zoff}" rpy="1.5707 0 -3.1414"/>
-    <limit upper="3.1415" lower="-3.1415" effort="30" velocity="5.0"/>
     <axis xyz="0 0 1"/>
-    <!-- <axis xyz="0 1 0"/> -->
   </joint>
   <!-- Caster wheel -->
@@ -224,5 +207,7 @@
       </geometry>
     </collision>
-    <xacro:sphere_inertia m="0.033" r="0.025"/>
+    <xacro:sphere_inertia mass="0.033" radius="0.025"/>
+      <origin xyz="0 0 0" rpy="0 0 0"/>
+    </xacro>
   </link>
   <joint name="caster_wheel_joint" type="fixed">
@@ -232,55 +217,3 @@
     <axis xyz="0 0 1"/>
   </joint>
-  <!-- Rplidar top -->
-  <link name="lidar_link">
-    <visual>
-      <geometry>
-        <mesh filename="package://real_lidarbot/models/lidarbot_description/meshes/rplidar_top.dae"/>
-      </geometry>
-    </visual>
-    <collision>
-      <origin xyz="0 -0.0009 0.011" rpy="0 0 0"/>
-      <geometry>
-        <cylinder radius="0.037" length="0.021"/>
-      </geometry>
-    </collision>
-  </link>
-  <joint name="lidar_joint" type="fixed">
-    <parent link="base_link"/>
-    <child link="lidar_link"/>
-    <origin xyz="0.0335 0.0095 0.069" rpy="0 0 0"/>
-    <axis xyz="0 0 1"/>
-  </joint>
-  <!-- Imu sensor  -->
-  <link name="imu_link">
-    <visual name="imu_visual">
-      <geometry>
-        <mesh filename="package://real_lidarbot/models/lidarbot_description/meshes/MPU6050.dae"/>
-      </geometry>
-    </visual>
-  </link>
-  <joint name="imu_joint" type="fixed">
-    <parent link="base_link"/>
-    <child link="imu_link"/>
-    <origin xyz="-0.06 0 0.0175" rpy="0 0 3.1414"/>
-  </joint>
-  <!-- Depth camera -->
-  <link name="camera_link">
-    <visual>
-      <geometry>
-        <mesh filename="package://real_lidarbot/models/lidarbot_description/meshes/d415.dae"/>
-      </geometry>
-    </visual>
-    <collision>
-      <origin xyz="0 0 -0.01" rpy="0 0 0"/>
-      <geometry>
-        <box size="0.1 0.025 0.022"/>
-      </geometry>
-    </collision>
-  </link>
-  <joint name="camera_joint" type="fixed">
-    <parent link="base_link"/>
-    <child link="camera_link"/>
-    <origin xyz="0.1 0 0.0425" rpy="1.5707 0 1.5707"/>
-  </joint>
 </robot>

Commit message: Changes to lidarbot_core.xacro

File: models/lidarbot_core.xacro (robot description, xacro)
@@ -10,5 +10,5 @@
   <xacro:property name="wheel_outer_radius" value="0.0325"/>
   <xacro:property name="wheel_inner_radius" value="0.0225"/>
-  <xacro:property name="wheel_width" value="0.025"/>
+  <xacro:property name="wheel_height" value="0.025"/>
   <!-- x-axis points forward, y-axis points to left, z-axis points upwards -->
   <!-- Define the gap between the wheel and chassis along y-axis in meters -->
@@ -157,8 +157,8 @@
       <origin xyz="0 0 0.0155" rpy="0 0 0"/>
       <geometry>
-        <cylinder radius="${wheel_outer_radius+0.01}" length="${wheel_width}"/>
-      </geometry>
-    </collision>
-    <xacro:thick_walled_cylinder_inertia m="0.031" outer_radius="${wheel_outer_radius}" inner_radius="${wheel_inner_radius}" h="${wheel_width}">
+        <cylinder radius="${wheel_outer_radius+0.01}" length="${wheel_height}"/>
+      </geometry>
+    </collision>
+    <xacro:thick_walled_cylinder_inertia mass="0.031" outer_radius="${wheel_outer_radius}" inner_radius="${wheel_inner_radius}" height="${wheel_height}">
       <origin xyz="0 0 0" rpy="0 0 0"/>
     </xacro>
@@ -181,8 +181,8 @@
       <origin xyz="0 0 -0.0065" rpy="0 0 0"/>
       <geometry>
-        <cylinder radius="${wheel_outer_radius+0.01}" length="${wheel_width}"/>
-      </geometry>
-    </collision>
-    <xacro:thick_walled_cylinder_inertia m="0.031" outer_radius="${wheel_outer_radius}" inner_radius="${wheel_inner_radius}" h="${wheel_width}">
+        <cylinder radius="${wheel_outer_radius+0.01}" length="${wheel_height}"/>
+      </geometry>
+    </collision>
+    <xacro:thick_walled_cylinder_inertia mass="0.031" outer_radius="${wheel_outer_radius}" inner_radius="${wheel_inner_radius}" height="${wheel_height}">
       <origin xyz="0 0 0" rpy="0 0 0"/>
     </xacro>

Commit message: Minor changes to lidarbot_core.xacro

File: models/lidarbot_core.xacro (robot description, xacro)
@@ -142,7 +142,7 @@
       </geometry>
     </collision>
-      <xacro:box_inertia mass="0.863" width="${base_width}" depth="${base_length}" height="${base_height}">
+      <!-- <xacro:box_inertia mass="0.863" width="${base_width}" depth="${base_length}" height="${base_height}">
         <origin xyz="0 0 -0.0125" rpy="0 0 0"/>
-      </xacro>
+      </xacro> -->
   </link>
   <!-- Left Wheel Link -->
@@ -160,7 +160,7 @@
       </geometry>
     </collision>
-    <xacro:thick_walled_cylinder_inertia mass="0.031" outer_radius="${wheel_outer_radius}" inner_radius="${wheel_inner_radius}" height="${wheel_height}">
-      <origin xyz="0 0 0" rpy="0 0 0"/>
-    </xacro>
+    <!-- <xacro:thick_walled_cylinder_inertia mass="0.031" outer_radius="${wheel_outer_radius}" inner_radius="${wheel_inner_radius}" height="${wheel_height}">
+      <origin xyz="0 0 0" rpy="0 0 0"/>
+    </xacro> -->
   </link>
   <joint name="left_wheel_joint" type="continuous">
@@ -184,7 +184,7 @@
       </geometry>
     </collision>
-    <xacro:thick_walled_cylinder_inertia mass="0.031" outer_radius="${wheel_outer_radius}" inner_radius="${wheel_inner_radius}" height="${wheel_height}">
-      <origin xyz="0 0 0" rpy="0 0 0"/>
-    </xacro>
+    <!-- <xacro:thick_walled_cylinder_inertia mass="0.031" outer_radius="${wheel_outer_radius}" inner_radius="${wheel_inner_radius}" height="${wheel_height}">
+      <origin xyz="0 0 0" rpy="0 0 0"/>
+    </xacro> -->
   </link>
   <joint name="right_wheel_joint" type="continuous">
@@ -207,7 +207,7 @@
       </geometry>
     </collision>
-    <xacro:sphere_inertia mass="0.033" radius="0.025"/>
-      <origin xyz="0 0 0" rpy="0 0 0"/>
-    </xacro>
+    <!-- <xacro:sphere_inertia mass="0.033" radius="0.025"/>
+      <origin xyz="0 0 0" rpy="0 0 0"/>
+    </xacro> -->
   </link>
   <joint name="caster_wheel_joint" type="fixed">

Commit message: Filled out closing xacro inertia tags

File: models/lidarbot_core.xacro (robot description, xacro)
@@ -2,5 +2,5 @@
 <robot xmlns:xacro="http://ros.org/wiki/xacro">
   <xacro:include filename="inertial_macros.xacro"/>
-  <!-- Robot constants -->
+  <!-- Robot constants (measurements in metres) -->
   <!-- Define the size of the robot's main chassis in meters-->
   <xacro:property name="base_length" value="0.21"/>
@@ -142,7 +142,7 @@
       </geometry>
     </collision>
-      <!-- <xacro:box_inertia mass="0.863" width="${base_width}" depth="${base_length}" height="${base_height}">
+      <xacro:box_inertia mass="0.863" width="${base_width}" depth="${base_length}" height="${base_height}">
         <origin xyz="0 0 -0.0125" rpy="0 0 0"/>
-      </xacro> -->
+      </xacro:box_inertia>
   </link>
   <!-- Left Wheel Link -->
@@ -162,5 +162,5 @@
     <xacro:thick_walled_cylinder_inertia mass="0.031" outer_radius="${wheel_outer_radius}" inner_radius="${wheel_inner_radius}" height="${wheel_height}">
       <origin xyz="0 0 0" rpy="0 0 0"/>
-    </xacro>
+    </xacro:thick_walled_cylinder_inertia>
   </link>
   <joint name="left_wheel_joint" type="continuous">
@@ -186,5 +186,5 @@
     <xacro:thick_walled_cylinder_inertia mass="0.031" outer_radius="${wheel_outer_radius}" inner_radius="${wheel_inner_radius}" height="${wheel_height}">
       <origin xyz="0 0 0" rpy="0 0 0"/>
-    </xacro>
+    </xacro:thick_walled_cylinder_inertia>
   </link>
   <joint name="right_wheel_joint" type="continuous">
@@ -207,7 +207,7 @@
       </geometry>
     </collision>
-    <!-- <xacro:sphere_inertia mass="0.033" radius="0.025"/>
-      <origin xyz="0 0 0" rpy="0 0 0"/>
-    </xacro> -->
+    <xacro:sphere_inertia mass="0.033" radius="0.025"/>
+      <origin xyz="0 0 0" rpy="0 0 0"/>
+  </xacro:sphere_inertia>
   </link>
   <joint name="caster_wheel_joint" type="fixed">

Commit message: Made minor correction in one of the inertial xacro tags

File: models/lidarbot_core.xacro (robot description, xacro)
@@ -19,5 +19,4 @@
   <!-- Defines the centre of the main robot chassis projected on the ground -->
   <link name="base_footprint"/>
-  <!-- The base footprint of the robot is located underneath the chassis/robot base  -->
   <joint name="base_joint" type="fixed">
     <parent link="base_footprint"/>
@@ -142,7 +141,7 @@
       </geometry>
     </collision>
-      <xacro:box_inertia mass="0.863" width="${base_width}" depth="${base_length}" height="${base_height}">
-        <origin xyz="0 0 -0.0125" rpy="0 0 0"/>
-      </xacro:box_inertia>
+    <xacro:box_inertia mass="0.863" width="${base_width}" depth="${base_length}" height="${base_height}">
+      <origin xyz="0 0 -0.0125" rpy="0 0 0"/>
+    </xacro:box_inertia>
   </link>
   <!-- Left Wheel Link -->
@@ -207,7 +206,7 @@
       </geometry>
     </collision>
-    <xacro:sphere_inertia mass="0.033" radius="0.025"/>
-      <origin xyz="0 0 0" rpy="0 0 0"/>
-  </xacro:sphere_inertia>
+    <xacro:sphere_inertia mass="0.033" radius="0.025">
+      <origin xyz="0 0 0" rpy="0 0 0"/>
+    </xacro:sphere_inertia>
   </link>
   <joint name="caster_wheel_joint" type="fixed">

Commit message: Adjusted base_joint origin

File: models/lidarbot_core.xacro (robot description, xacro)
@@ -21,5 +21,6 @@
     <parent link="base_footprint"/>
     <child link="base_link"/>
-    <origin xyz="0 0 ${(wheel_outer_radius+wheel_zoff)}" rpy="0 0 0"/>
+    <origin xyz="0 0 0" rpy="0 0 0"/>
+    <!-- <origin xyz="0 0 ${(wheel_outer_radius+wheel_zoff)}" rpy="0 0 0"/> -->
   </joint>
   <!-- Robot Base -->

Commit message: Adjusted base_joint origin

File: models/lidarbot_core.xacro (robot description, xacro)
@@ -21,11 +21,12 @@
     <parent link="base_footprint"/>
     <child link="base_link"/>
-    <origin xyz="0 0 0" rpy="0 0 0"/>
-    <!-- <origin xyz="0 0 ${(wheel_outer_radius+wheel_zoff)}" rpy="0 0 0"/> -->
+    <!-- <origin xyz="0 0 0" rpy="0 0 0"/> -->
+    <origin xyz="0 0 ${(wheel_outer_radius+wheel_zoff)}" rpy="0 0 0"/>
   </joint>
   <!-- Robot Base -->
   <link name="base_link">
       <visual>
-        <origin xyz="0 0 -0.0125" rpy="0 0 0"/>
+        <origin xyz="0 0 0" rpy="0 0 0"/>
+        <!-- <origin xyz="0 0 -0.0125" rpy="0 0 0"/> -->
           <geometry>
               <mesh filename="package://real_lidarbot/models/lidarbot_description/meshes/robot_base_link.dae" />

Commit message: Adjusted base_joint origin

File: models/lidarbot_core.xacro (robot description, xacro)
@@ -27,5 +27,5 @@
   <link name="base_link">
       <visual>
-        <origin xyz="0 0 0" rpy="0 0 0"/>
+        <origin xyz="0 0 ${(wheel_outer_radius+wheel_zoff)}" rpy="0 0 0"/>
         <!-- <origin xyz="0 0 -0.0125" rpy="0 0 0"/> -->
           <geometry>

Commit message: Adjusted base_joint origin

File: models/lidarbot_core.xacro (robot description, xacro)
@@ -21,6 +21,6 @@
     <parent link="base_footprint"/>
     <child link="base_link"/>
-    <!-- <origin xyz="0 0 0" rpy="0 0 0"/> -->
-    <origin xyz="0 0 ${(wheel_outer_radius+wheel_zoff)}" rpy="0 0 0"/>
+    <origin xyz="0 0 0" rpy="0 0 0"/>
+    <!-- <origin xyz="0 0 ${(wheel_outer_radius+wheel_zoff)}" rpy="0 0 0"/> -->
   </joint>
   <!-- Robot Base -->

Commit message: Adjusted base_joint origin

File: models/lidarbot_core.xacro (robot description, xacro)
@@ -21,11 +21,12 @@
     <parent link="base_footprint"/>
     <child link="base_link"/>
-    <origin xyz="0 0 0" rpy="0 0 0"/>
-    <!-- <origin xyz="0 0 ${(wheel_outer_radius+wheel_zoff)}" rpy="0 0 0"/> -->
+    <!-- <origin xyz="0 0 0" rpy="0 0 0"/> -->
+    <origin xyz="0 0 ${(wheel_outer_radius+wheel_zoff)}" rpy="0 0 0"/>
   </joint>
   <!-- Robot Base -->
   <link name="base_link">
       <visual>
-        <origin xyz="0 0 ${(wheel_outer_radius+wheel_zoff)}" rpy="0 0 0"/>
+        <origin xyz="${base_length/2} 0 ${base_height}" rpy="0 0 0"/>
+        <!-- <origin xyz="0 0 ${(wheel_outer_radius+wheel_zoff)}" rpy="0 0 0"/> -->
         <!-- <origin xyz="0 0 -0.0125" rpy="0 0 0"/> -->
           <geometry>

Commit message: Adjusted base_joint origin

File: models/lidarbot_core.xacro (robot description, xacro)
@@ -27,5 +27,5 @@
   <link name="base_link">
       <visual>
-        <origin xyz="${base_length/2} 0 ${base_height}" rpy="0 0 0"/>
+        <origin xyz="0 0 ${base_height}" rpy="0 0 0"/>
         <!-- <origin xyz="0 0 ${(wheel_outer_radius+wheel_zoff)}" rpy="0 0 0"/> -->
         <!-- <origin xyz="0 0 -0.0125" rpy="0 0 0"/> -->

Commit message: Made changes to wheel joint types in model.sdf

File: models/lidarbot_core.xacro (robot description, xacro)
@@ -27,7 +27,7 @@
   <link name="base_link">
       <visual>
-        <origin xyz="0 0 ${base_height}" rpy="0 0 0"/>
+        <!-- <origin xyz="0 0 ${base_height}" rpy="0 0 0"/> -->
         <!-- <origin xyz="0 0 ${(wheel_outer_radius+wheel_zoff)}" rpy="0 0 0"/> -->
-        <!-- <origin xyz="0 0 -0.0125" rpy="0 0 0"/> -->
+        <origin xyz="0 0 -0.0125" rpy="0 0 0"/>
           <geometry>
               <mesh filename="package://real_lidarbot/models/lidarbot_description/meshes/robot_base_link.dae" />

Commit message: Changes to core xacro file

File: models/lidarbot_core.xacro (robot description, xacro)
@@ -27,5 +27,5 @@
         <!-- <origin xyz="0 0 ${base_height}" rpy="0 0 0"/> -->
         <!-- <origin xyz="0 0 ${(wheel_outer_radius+wheel_zoff)}" rpy="0 0 0"/> -->
-        <origin xyz="0 0 -0.0125" rpy="0 0 0"/>
+        <!-- <origin xyz="0 0 -0.0125" rpy="0 0 0"/> -->
           <geometry>
               <mesh filename="package://real_lidarbot/models/lidarbot_description/meshes/robot_base_link.dae" />

Commit message: Changes to core xacro file

File: models/lidarbot_core.xacro (robot description, xacro)
@@ -17,6 +17,6 @@
   <link name="base_footprint"/>
   <joint name="base_joint" type="fixed">
-    <parent link="base_footprint"/>
-    <child link="base_link"/>
+    <parent link="base_link"/>
+    <child link="base_footprint"/>
     <!-- <origin xyz="0 0 0" rpy="0 0 0"/> -->
     <origin xyz="0 0 ${-(wheel_outer_radius+wheel_zoff)}" rpy="0 0 0"/>

Commit message: Changes to core xacro file

File: models/lidarbot_core.xacro (robot description, xacro)
@@ -27,5 +27,5 @@
         <!-- <origin xyz="0 0 ${base_height}" rpy="0 0 0"/> -->
         <!-- <origin xyz="0 0 ${(wheel_outer_radius+wheel_zoff)}" rpy="0 0 0"/> -->
-        <!-- <origin xyz="0 0 -0.0125" rpy="0 0 0"/> -->
+        <origin xyz="0 0 -0.0125" rpy="0 0 0"/>
           <geometry>
               <mesh filename="package://real_lidarbot/models/lidarbot_description/meshes/robot_base_link.dae" />

Commit message: Changes to core xacro file

File: models/lidarbot_core.xacro (robot description, xacro)
@@ -25,7 +25,6 @@
   <link name="base_link">
       <visual>
-        <!-- <origin xyz="0 0 ${base_height}" rpy="0 0 0"/> -->
-        <!-- <origin xyz="0 0 ${(wheel_outer_radius+wheel_zoff)}" rpy="0 0 0"/> -->
-        <origin xyz="0 0 -0.0125" rpy="0 0 0"/>
+        <origin xyz="0 0 ${wheel_zoff}" rpy="0 0 0"/>
+        <!-- <origin xyz="0 0 ${-wheel_zoff}" rpy="0 0 0"/> -->
           <geometry>
               <mesh filename="package://real_lidarbot/models/lidarbot_description/meshes/robot_base_link.dae" />

Commit message: Changes to core xacro file

File: models/lidarbot_core.xacro (robot description, xacro)
@@ -17,13 +17,14 @@
   <link name="base_footprint"/>
   <joint name="base_joint" type="fixed">
-    <parent link="base_link"/>
-    <child link="base_footprint"/>
+    <parent link="base_footprint"/>
+    <child link="base_link"/>
     <!-- <origin xyz="0 0 0" rpy="0 0 0"/> -->
-    <origin xyz="0 0 ${-(wheel_outer_radius+wheel_zoff)}" rpy="0 0 0"/>
+    <origin xyz="0 0 ${(wheel_outer_radius+wheel_zoff)}" rpy="0 0 0"/>
+    <!-- <origin xyz="0 0 ${-(wheel_outer_radius+wheel_zoff)}" rpy="0 0 0"/> -->
   </joint>
   <!-- Robot Base -->
   <link name="base_link">
       <visual>
-        <origin xyz="0 0 ${wheel_zoff}" rpy="0 0 0"/>
+        <origin xyz="0 0 ${wheel_outer_radius+wheel_zoff}" rpy="0 0 0"/>
         <!-- <origin xyz="0 0 ${-wheel_zoff}" rpy="0 0 0"/> -->
           <geometry>
@@ -147,5 +148,5 @@
   <link name="left_wheel">
     <visual>
-      <origin xyz="0 0 0" rpy="0 0 0"/>
+      <!-- <origin xyz="0 0 0" rpy="0 0 0"/> -->
         <geometry>
           <mesh filename="package://real_lidarbot/models/lidarbot_description/meshes/left_wheel.dae" />
@@ -171,5 +172,5 @@
   <link name="right_wheel">
     <visual>
-      <origin xyz="0 0 0" rpy="0 0 0"/>
+      <!-- <origin xyz="0 0 0" rpy="0 0 0"/> -->
       <geometry>
         <mesh filename="package://real_lidarbot/models/lidarbot_description/meshes/right_wheel.dae"/>

Commit message: Changes to core xacro file

File: models/lidarbot_core.xacro (robot description, xacro)
@@ -26,5 +26,5 @@
   <link name="base_link">
       <visual>
-        <origin xyz="0 0 ${wheel_outer_radius+wheel_zoff}" rpy="0 0 0"/>
+        <!-- <origin xyz="0 0 ${wheel_outer_radius+wheel_zoff}" rpy="0 0 0"/> -->
         <!-- <origin xyz="0 0 ${-wheel_zoff}" rpy="0 0 0"/> -->
           <geometry>

Commit message: Changes to core xacro file

File: models/lidarbot_core.xacro (robot description, xacro)
@@ -27,5 +27,5 @@
       <visual>
         <!-- <origin xyz="0 0 ${wheel_outer_radius+wheel_zoff}" rpy="0 0 0"/> -->
-        <!-- <origin xyz="0 0 ${-wheel_zoff}" rpy="0 0 0"/> -->
+        <origin xyz="0 0 ${-wheel_zoff}" rpy="0 0 0"/>
           <geometry>
               <mesh filename="package://real_lidarbot/models/lidarbot_description/meshes/robot_base_link.dae" />

Commit message: Changes to core xacro file

File: models/lidarbot_core.xacro (robot description, xacro)
@@ -17,14 +17,12 @@
   <link name="base_footprint"/>
   <joint name="base_joint" type="fixed">
-    <parent link="base_footprint"/>
-    <child link="base_link"/>
-    <!-- <origin xyz="0 0 0" rpy="0 0 0"/> -->
-    <origin xyz="0 0 ${(wheel_outer_radius+wheel_zoff)}" rpy="0 0 0"/>
-    <!-- <origin xyz="0 0 ${-(wheel_outer_radius+wheel_zoff)}" rpy="0 0 0"/> -->
+    <parent link="base_link"/>
+    <child link="base_footprint"/>
+    <!-- <origin xyz="0 0 ${(wheel_outer_radius+wheel_zoff)}" rpy="0 0 0"/> -->
+    <origin xyz="0 0 ${-(wheel_outer_radius+wheel_zoff)}" rpy="0 0 0"/>
   </joint>
   <!-- Robot Base -->
   <link name="base_link">
       <visual>
-        <!-- <origin xyz="0 0 ${wheel_outer_radius+wheel_zoff}" rpy="0 0 0"/> -->
         <origin xyz="0 0 ${-wheel_zoff}" rpy="0 0 0"/>
           <geometry>
