Commit message: Changes to core xacro file

File: models/lidarbot_core.xacro (robot description, xacro)
@@ -10,6 +10,4 @@
   <xacro:property name="wheel_inner_radius" value="0.0225"/>
   <xacro:property name="wheel_height" value="0.025"/>
-  <!-- Gap between the wheel and chassis along y-axis -->
-  <xacro:property name="wheel_ygap" value="0.003"/>
   <!-- Distance between centre of wheel and robot base/chassis -->
   <xacro:property name="wheel_zoff" value="0.0125"/>
@@ -19,5 +17,4 @@
     <parent link="base_link"/>
     <child link="base_footprint"/>
-    <!-- <origin xyz="0 0 ${(wheel_outer_radius+wheel_zoff)}" rpy="0 0 0"/> -->
     <origin xyz="0 0 ${-(wheel_outer_radius+wheel_zoff)}" rpy="0 0 0"/>
   </joint>
@@ -48,95 +45,95 @@
         </geometry>
       </collision>
-     <!-- Rpi stand -->
-     <visual name="rpi_4_stand_visual">
-      <origin xyz="-0.06 0.015 0.031" rpy="${pi} 0 ${-pi}"/>
-        <geometry>
-            <mesh filename="package://real_lidarbot/models/lidarbot_description/meshes/rpi_stand.dae" />
-        </geometry>
-    </visual>
-    <collision name="rpi_4_stand_collision">
-      <origin xyz="-0.06 0 0.017" rpy="0 0 ${pi/2}"/>
-      <geometry>
-        <box size="0.098 0.065 0.034"/>
-      </geometry>
-    </collision>
-    <!-- Raspberry Pi -->
-    <visual name="rpi_4_visual">
-      <origin xyz="-0.059 0.00245 0.033" rpy="0 0 ${pi/2}"/>
-      <geometry>
-        <mesh filename="package://real_lidarbot/models/lidarbot_description/meshes/rpi_4.dae"/>
-      </geometry>
-    </visual>
-    <collision name="rpi_4_collision">
-      <origin xyz="-0.058 0.005 0.041" rpy="0 0 ${pi/2}"/>
-      <geometry>
-        <box size="0.09 0.06 0.02"/>
-      </geometry>
-    </collision>
-    <!-- Power bank stand -->
-    <visual name="power_bank_stand_visual">
-      <origin xyz="0.033 0.015 0.031" rpy="${pi} 0 ${pi}"/>
-      <geometry>
-        <mesh filename="package://real_lidarbot/models/lidarbot_description/meshes/power_bank_stand.dae"/>
-      </geometry>
-    </visual>
-    <collision name="power_bank_stand_collision">
-      <origin xyz="0.033 0 0.0085" rpy="0 0 ${pi/2}"/>
-      <geometry>
-        <box size="0.098 0.065 0.015"/>
-      </geometry>
-    </collision>
-    <!-- Power bank -->
-    <visual name="power_bank_visual">
-      <origin xyz="0.0635 0.04775 0.015" rpy="0 0 ${pi/2}"/>
-      <geometry>
-        <mesh filename="package://real_lidarbot/models/lidarbot_description/meshes/power_bank.dae"/>
-      </geometry>
-    </visual>
-    <collision name="power_bank_collision">
-      <origin xyz="0.033 0 0.025" rpy="0 0 ${pi/2}"/>
-      <geometry>
-        <box size="0.096 0.062 0.02"/>
-      </geometry>
-    </collision>
-    <!-- Rplidar stand -->
-    <visual name="rplidar_stand_visual">
-      <origin xyz="0.033 0.015 0.017" rpy="0 0 ${-2*pi}"/>
-      <geometry>
-        <mesh filename="package://real_lidarbot/models/lidarbot_description/meshes/rplidar_stand.dae"/>
-      </geometry>
-    </visual>
-    <collision name="rplidar_stand_collision">
-      <origin xyz="0.033 0 0.04" rpy="0 0 ${pi/2}"/>
-      <geometry>
-        <box size="0.098 0.065 0.015"/>
-      </geometry>
-    </collision>
-    <!-- Rplidar base -->
-    <visual name="rplidar_base_visual">
-      <origin xyz="0.03485 0.0087 0.037" rpy="0 0 ${-pi/2}"/>
-        <geometry>
-          <mesh filename="package://real_lidarbot/models/lidarbot_description/meshes/rplidar_base.dae"/>
-        </geometry>
-      </visual>
-    <collision name="rplidar_base_collision">
-      <origin xyz="0.033 0 0.056" rpy="0 0 ${-pi/2}"/>
-      <geometry>
-        <box size="0.12 0.072 0.035"/>
-      </geometry>
-    </collision>
-    <!-- Depth camera mount -->
-    <visual name="camera_mount_visual">
-      <origin xyz="0.089 0 0.016" rpy="0 0 0"/>
-        <geometry>
-          <cylinder radius="0.007" length="0.03"/>
-        </geometry>
-    </visual>
-    <collision name="camera_mount_collision">
-      <origin xyz="0.089 0 0.016" rpy="0 0 0"/>
-      <geometry>
-        <cylinder radius="0.008" length="0.031"/>
-      </geometry>
-    </collision>
+      <!-- Rpi stand -->
+      <visual name="rpi_4_stand_visual">
+        <origin xyz="-0.06 0.015 0.031" rpy="${pi} 0 ${-pi}"/>
+          <geometry>
+              <mesh filename="package://real_lidarbot/models/lidarbot_description/meshes/rpi_stand.dae" />
+          </geometry>
+      </visual>
+      <collision name="rpi_4_stand_collision">
+        <origin xyz="-0.06 0 0.017" rpy="0 0 ${pi/2}"/>
+        <geometry>
+          <box size="0.098 0.065 0.034"/>
+        </geometry>
+      </collision>
+      <!-- Raspberry Pi -->
+      <visual name="rpi_4_visual">
+        <origin xyz="-0.059 0.00245 0.033" rpy="0 0 ${pi/2}"/>
+        <geometry>
+          <mesh filename="package://real_lidarbot/models/lidarbot_description/meshes/rpi_4.dae"/>
+        </geometry>
+      </visual>
+      <collision name="rpi_4_collision">
+        <origin xyz="-0.058 0.005 0.041" rpy="0 0 ${pi/2}"/>
+        <geometry>
+          <box size="0.09 0.06 0.02"/>
+        </geometry>
+      </collision>
+      <!-- Power bank stand -->
+      <visual name="power_bank_stand_visual">
+        <origin xyz="0.033 0.015 0.031" rpy="${pi} 0 ${pi}"/>
+        <geometry>
+          <mesh filename="package://real_lidarbot/models/lidarbot_description/meshes/power_bank_stand.dae"/>
+        </geometry>
+      </visual>
+      <collision name="power_bank_stand_collision">
+        <origin xyz="0.033 0 0.0085" rpy="0 0 ${pi/2}"/>
+        <geometry>
+          <box size="0.098 0.065 0.015"/>
+        </geometry>
+      </collision>
+      <!-- Power bank -->
+      <visual name="power_bank_visual">
+        <origin xyz="0.0635 0.04775 0.015" rpy="0 0 ${pi/2}"/>
+        <geometry>
+          <mesh filename="package://real_lidarbot/models/lidarbot_description/meshes/power_bank.dae"/>
+        </geometry>
+      </visual>
+      <collision name="power_bank_collision">
+        <origin xyz="0.033 0 0.025" rpy="0 0 ${pi/2}"/>
+        <geometry>
+          <box size="0.096 0.062 0.02"/>
+        </geometry>
+      </collision>
+      <!-- Rplidar stand -->
+      <visual name="rplidar_stand_visual">
+        <origin xyz="0.033 0.015 0.017" rpy="0 0 ${-2*pi}"/>
+        <geometry>
+          <mesh filename="package://real_lidarbot/models/lidarbot_description/meshes/rplidar_stand.dae"/>
+        </geometry>
+      </visual>
+      <collision name="rplidar_stand_collision">
+        <origin xyz="0.033 0 0.04" rpy="0 0 ${pi/2}"/>
+        <geometry>
+          <box size="0.098 0.065 0.015"/>
+        </geometry>
+      </collision>
+      <!-- Rplidar base -->
+      <visual name="rplidar_base_visual">
+        <origin xyz="0.03485 0.0087 0.037" rpy="0 0 ${-pi/2}"/>
+          <geometry>
+            <mesh filename="package://real_lidarbot/models/lidarbot_description/meshes/rplidar_base.dae"/>
+          </geometry>
+        </visual>
+      <collision name="rplidar_base_collision">
+        <origin xyz="0.033 0 0.056" rpy="0 0 ${-pi/2}"/>
+        <geometry>
+          <box size="0.12 0.072 0.035"/>
+        </geometry>
+      </collision>
+      <!-- Depth camera mount -->
+      <visual name="camera_mount_visual">
+        <origin xyz="0.089 0 0.016" rpy="0 0 0"/>
+          <geometry>
+            <cylinder radius="0.007" length="0.03"/>
+          </geometry>
+      </visual>
+      <collision name="camera_mount_collision">
+        <origin xyz="0.089 0 0.016" rpy="0 0 0"/>
+        <geometry>
+          <cylinder radius="0.008" length="0.031"/>
+        </geometry>
+      </collision>
     <xacro:box_inertia mass="0.864" length="${base_length}" width="${base_width}" height="${base_height}">
       <origin xyz="0 0 -0.0125" rpy="0 0 0"/>
@@ -146,5 +143,4 @@
   <link name="left_wheel">
     <visual>
-      <!-- <origin xyz="0 0 0" rpy="0 0 0"/> -->
         <geometry>
           <mesh filename="package://real_lidarbot/models/lidarbot_description/meshes/left_wheel.dae" />
@@ -170,5 +166,4 @@
   <link name="right_wheel">
     <visual>
-      <!-- <origin xyz="0 0 0" rpy="0 0 0"/> -->
       <geometry>
         <mesh filename="package://real_lidarbot/models/lidarbot_description/meshes/right_wheel.dae"/>
@@ -188,5 +183,5 @@
     <parent link="base_link"/>
     <child link="right_wheel"/>
-    <origin xyz="-0.028 -0.065 -${wheel_zoff}" rpy="${pi/2} 0 ${-pi}"/>
+    <origin xyz="-0.028 -0.065 -${wheel_zoff}" rpy="${-pi/2} 0 ${-pi}"/>
     <axis xyz="0 0 1"/>
   </joint>

Commit message: Changes to core xacro file

File: models/lidarbot_core.xacro (robot description, xacro)
@@ -183,5 +183,5 @@
     <parent link="base_link"/>
     <child link="right_wheel"/>
-    <origin xyz="-0.028 -0.065 -${wheel_zoff}" rpy="${-pi/2} 0 ${-pi}"/>
+    <origin xyz="-0.028 -0.065 -${wheel_zoff}" rpy="${pi/2} 0 ${-pi}"/>
     <axis xyz="0 0 1"/>
   </joint>

Commit message: Made some adjustments to core xacro file

File: models/lidarbot_core.xacro (robot description, xacro)
@@ -173,5 +173,5 @@
       <origin xyz="0 0 -0.0065" rpy="0 0 0"/>
       <geometry>
-        <cylinder radius="${wheel_outer_radius+0.01}" length="${wheel_height}"/>
+        <cylinder radius="${wheel_outer_radius}" length="${wheel_height}"/>
       </geometry>
     </collision>

Commit message: Made some adjustments to core xacro file

File: models/lidarbot_core.xacro (robot description, xacro)
@@ -150,5 +150,6 @@
       <origin xyz="0 0 0.0155" rpy="0 0 0"/>
       <geometry>
-        <cylinder radius="${wheel_outer_radius+0.01}" length="${wheel_height}"/>
+        <cylinder radius="${wheel_outer_radius}" length="${wheel_height}"/>
+        <!-- <cylinder radius="${wheel_outer_radius+0.01}" length="${wheel_height}"/> -->
       </geometry>
     </collision>
@@ -174,4 +175,5 @@
       <geometry>
         <cylinder radius="${wheel_outer_radius}" length="${wheel_height}"/>
+        <!-- <cylinder radius="${wheel_outer_radius+0.01}" length="${wheel_height}"/> -->
       </geometry>
     </collision>

Commit message: Made some adjustments to core xacro file

File: models/lidarbot_core.xacro (robot description, xacro)
@@ -150,6 +150,6 @@
       <origin xyz="0 0 0.0155" rpy="0 0 0"/>
       <geometry>
-        <cylinder radius="${wheel_outer_radius}" length="${wheel_height}"/>
-        <!-- <cylinder radius="${wheel_outer_radius+0.01}" length="${wheel_height}"/> -->
+        <!-- <cylinder radius="${wheel_outer_radius}" length="${wheel_height}"/> -->
+        <cylinder radius="${wheel_outer_radius+0.01}" length="${wheel_height}"/>
       </geometry>
     </collision>
@@ -174,6 +174,6 @@
       <origin xyz="0 0 -0.0065" rpy="0 0 0"/>
       <geometry>
-        <cylinder radius="${wheel_outer_radius}" length="${wheel_height}"/>
-        <!-- <cylinder radius="${wheel_outer_radius+0.01}" length="${wheel_height}"/> -->
+        <!-- <cylinder radius="${wheel_outer_radius}" length="${wheel_height}"/> -->
+        <cylinder radius="${wheel_outer_radius+0.01}" length="${wheel_height}"/>
       </geometry>
     </collision>

Commit message: Edits to core xacro file

File: models/lidarbot_core.xacro (robot description, xacro)
@@ -150,6 +150,5 @@
       <origin xyz="0 0 0.0155" rpy="0 0 0"/>
       <geometry>
-        <!-- <cylinder radius="${wheel_outer_radius}" length="${wheel_height}"/> -->
-        <cylinder radius="${wheel_outer_radius+0.01}" length="${wheel_height}"/>
+        <cylinder radius="${wheel_outer_radius}" length="${wheel_height}"/>
       </geometry>
     </collision>
@@ -174,6 +173,5 @@
       <origin xyz="0 0 -0.0065" rpy="0 0 0"/>
       <geometry>
-        <!-- <cylinder radius="${wheel_outer_radius}" length="${wheel_height}"/> -->
-        <cylinder radius="${wheel_outer_radius+0.01}" length="${wheel_height}"/>
+        <cylinder radius="${wheel_outer_radius}" length="${wheel_height}"/>
       </geometry>
     </collision>

Commit message: Minor change in core xacro file

File: models/lidarbot_core.xacro (robot description, xacro)
@@ -15,7 +15,8 @@
   <link name="base_footprint"/>
   <joint name="base_joint" type="fixed">
-    <parent link="base_link"/>
-    <child link="base_footprint"/>
-    <origin xyz="0 0 ${-(wheel_outer_radius+wheel_zoff)}" rpy="0 0 0"/>
+    <parent link="base_footprint"/>
+    <child link="base_link"/>
+    <origin xyz="0 0 ${(wheel_outer_radius+wheel_zoff)}" rpy="0 0 0"/>
+    <!-- <origin xyz="0 0 ${-(wheel_outer_radius+wheel_zoff)}" rpy="0 0 0"/> -->
   </joint>
   <!-- Robot Base -->

Commit message: Minor change in core xacro file

File: models/lidarbot_core.xacro (robot description, xacro)
@@ -18,5 +18,4 @@
     <child link="base_link"/>
     <origin xyz="0 0 ${(wheel_outer_radius+wheel_zoff)}" rpy="0 0 0"/>
-    <!-- <origin xyz="0 0 ${-(wheel_outer_radius+wheel_zoff)}" rpy="0 0 0"/> -->
   </joint>
   <!-- Robot Base -->
@@ -191,5 +190,6 @@
     <visual>
       <geometry>
-        <mesh filename="package://real_lidarbot/models/lidarbot_description/meshes/caster_wheel.dae"/>
+        <mesh filename="package://models/lidarbot_description/meshes/caster_wheel.dae"/>
+        <!-- <mesh filename="package://real_lidarbot/models/lidarbot_description/meshes/caster_wheel.dae"/> -->
       </geometry>
     </visual>

Commit message: Testing out changes to robot_state_publisher_launch.py

File: models/lidarbot_core.xacro (robot description, xacro)
@@ -214,5 +214,4 @@
     <child link="caster_wheel"/>
     <origin xyz="0.0925 0 -0.031" rpy="0 0 ${pi/2}"/>
-    <axis xyz="0 0 1"/>
   </joint>
 </robot>

Commit message: Changes to core xacro

File: models/lidarbot_core.xacro (robot description, xacro)
@@ -161,5 +161,5 @@
     </xacro:cylinder_inertia>
   </link>
-  <joint name="left_wheel_joint" type="continuous">
+  <joint name="left_wheel_joint" type="revolute">
     <parent link="base_link"/>
     <child link="left_wheel"/>
@@ -187,5 +187,5 @@
     </xacro:cylinder_inertia>
   </link>
-  <joint name="right_wheel_joint" type="continuous">
+  <joint name="right_wheel_joint" type="revolute">
     <parent link="base_link"/>
     <child link="right_wheel"/>

Commit message: Changes to core xacro

File: models/lidarbot_core.xacro (robot description, xacro)
@@ -187,5 +187,5 @@
     </xacro:cylinder_inertia>
   </link>
-  <joint name="right_wheel_joint" type="revolute">
+  <joint name="right_wheel_joint" type="continuous">
     <parent link="base_link"/>
     <child link="right_wheel"/>

Commit message: Changes to core xacro

File: models/lidarbot_core.xacro (robot description, xacro)
@@ -161,5 +161,5 @@
     </xacro:cylinder_inertia>
   </link>
-  <joint name="left_wheel_joint" type="revolute">
+  <joint name="left_wheel_joint" type="continuous">
     <parent link="base_link"/>
     <child link="left_wheel"/>
@@ -187,4 +187,5 @@
     </xacro:cylinder_inertia>
   </link>
+  <!-- Stopped here -->
   <joint name="right_wheel_joint" type="continuous">
     <parent link="base_link"/>

Commit message: Changes to core xacro and model.sdf

File: models/lidarbot_core.xacro (robot description, xacro)
@@ -161,8 +161,9 @@
     </xacro:cylinder_inertia>
   </link>
-  <joint name="left_wheel_joint" type="continuous">
+  <joint name="left_wheel_joint" type="revolute">
     <parent link="base_link"/>
     <child link="left_wheel"/>
     <origin xyz="-0.028 0.055 -${wheel_zoff}" rpy="${pi/2} 0 ${pi}"/>
+    <limit upper="3.1415" lower="-3.1415" effort="30" velocity="5.0"/>
     <axis xyz="0 0 1"/>
   </joint>
@@ -188,8 +189,9 @@
   </link>
   <!-- Stopped here -->
-  <joint name="right_wheel_joint" type="continuous">
+  <joint name="right_wheel_joint" type="revolute">
     <parent link="base_link"/>
     <child link="right_wheel"/>
     <origin xyz="-0.028 -0.065 -${wheel_zoff}" rpy="${pi/2} 0 ${-pi}"/>
+    <limit upper="3.1415" lower="-3.1415" effort="30" velocity="5.0"/>
     <axis xyz="0 0 1"/>
   </joint>

Commit message: Files renamed

File: models/lidarbot_core.xacro (robot description, xacro)
@@ -25,6 +25,6 @@
         <origin xyz="0 0 ${-wheel_zoff}" rpy="0 0 0"/>
           <geometry>
-              <mesh filename="package://real_lidarbot/models/lidarbot_description/meshes/robot_base_link.dae" />
-          </geometry>
+              <mesh filename="package://real_lidarbot/models/lidarbot_description/meshes/robot_base.dae" />
+          </geometryk>
       </visual>
       <collision>

Commit message: File renames

File: models/lidarbot_core.xacro (robot description, xacro)
@@ -25,5 +25,5 @@
         <origin xyz="0 0 ${-wheel_zoff}" rpy="0 0 0"/>
           <geometry>
-              <mesh filename="package://real_lidarbot/models/lidarbot_description/meshes/robot_base.dae" />
+              <mesh filename="package://real_lidarbot/models/lidarbot_description/meshes/robot_base_link.dae" />
           </geometryk>
       </visual>

Commit message: adjusting file directories for geometry meshes

File: models/lidarbot_core.xacro (robot description, xacro)
@@ -25,5 +25,6 @@
         <origin xyz="0 0 ${-wheel_zoff}" rpy="0 0 0"/>
           <geometry>
-              <mesh filename="package://real_lidarbot/models/lidarbot_description/meshes/robot_base.dae" />
+              <mesh filename="lidarbot_description/meshes/robot_base.dae" />
+              <!-- <mesh filename="package://real_lidarbot/models/lidarbot_description/meshes/robot_base.dae" /> -->
           </geometry>
       </visual>

Commit message: Changed wheel joint type to continuous

File: models/lidarbot_core.xacro (robot description, xacro)
@@ -159,9 +159,9 @@
     </xacro:cylinder_inertia>
   </link>
-  <joint name="left_wheel_joint" type="revolute">
+  <joint name="left_wheel_joint" type="continuous">
     <parent link="base_link"/>
     <child link="left_wheel"/>
     <origin xyz="-0.028 0.055 -${wheel_zoff}" rpy="${pi/2} 0 ${pi}"/>
-    <limit upper="3.1415" lower="-3.1415" effort="30" velocity="5.0"/>
+    <!-- <limit upper="3.1415" lower="-3.1415" effort="30" velocity="5.0"/> -->
     <axis xyz="0 0 1"/>
   </joint>
@@ -183,9 +183,9 @@
     </xacro:cylinder_inertia>
   </link>
-  <joint name="right_wheel_joint" type="revolute">
+  <joint name="right_wheel_joint" type="continuous">
     <parent link="base_link"/>
     <child link="right_wheel"/>
     <origin xyz="-0.028 -0.065 -${wheel_zoff}" rpy="${pi/2} 0 ${-pi}"/>
-    <limit upper="3.1415" lower="-3.1415" effort="30" velocity="5.0"/>
+    <!-- <limit upper="3.1415" lower="-3.1415" effort="30" velocity="5.0"/> -->
     <axis xyz="0 0 1"/>
   </joint>

Commit message: Changed back location of robot_base mesh in lidarbot

File: models/lidarbot_core.xacro (robot description, xacro)
@@ -25,6 +25,6 @@
         <origin xyz="0 0 ${-wheel_zoff}" rpy="0 0 0"/>
           <geometry>
-              <mesh filename="lidarbot_description/meshes/robot_base.dae" />
-              <!-- <mesh filename="package://real_lidarbot/models/lidarbot_description/meshes/robot_base.dae" /> -->
+              <!-- <mesh filename="lidarbot_description/meshes/robot_base.dae" /> -->
+              <mesh filename="package://real_lidarbot/models/lidarbot_description/meshes/robot_base.dae" />
           </geometry>
       </visual>

Commit message: Adding mesh for robot base collision

File: models/lidarbot_core.xacro (robot description, xacro)
@@ -31,5 +31,6 @@
       <collision>
         <geometry>
-          <box size="${base_length} ${base_width} ${base_height}"/>
+          <!-- <box size="${base_length} ${base_width} ${base_height}"/> -->
+          <mesh filename="package://real_lidarbot/models/lidarbot_description/meshes/robot_base.dae" />
         </geometry>
       </collision>

Commit message: Trying out a new format for calling mesh files

File: models/lidarbot_core.xacro (robot description, xacro)
@@ -25,12 +25,11 @@
         <origin xyz="0 0 ${-wheel_zoff}" rpy="0 0 0"/>
           <geometry>
-              <!-- <mesh filename="lidarbot_description/meshes/robot_base.dae" /> -->
-              <mesh filename="package://real_lidarbot/models/lidarbot_description/meshes/robot_base.dae" />
+              <mesh filename="file://$(find real_lidarbot)/models/lidarbot_description/meshes/robot_base.dae" />
+              <!-- <mesh filename="package://real_lidarbot/models/lidarbot_description/meshes/robot_base.dae" /> -->
           </geometry>
       </visual>
       <collision>
         <geometry>
-          <!-- <box size="${base_length} ${base_width} ${base_height}"/> -->
-          <mesh filename="package://real_lidarbot/models/lidarbot_description/meshes/robot_base.dae" />
+          <box size="${base_length} ${base_width} ${base_height}"/>
         </geometry>
       </collision>

Commit message: Changed wheel collision geometry

File: models/lidarbot_core.xacro (robot description, xacro)
@@ -7,6 +7,5 @@
   <xacro:property name="base_height" value="0.035"/>
   <!-- Robot's wheel properties -->
-  <xacro:property name="wheel_outer_radius" value="0.0325"/>
-  <xacro:property name="wheel_inner_radius" value="0.0225"/>
+  <xacro:property name="wheel_radius" value="0.0325"/>
   <xacro:property name="wheel_height" value="0.025"/>
   <xacro:property name="wheel_mass" value="0.031"/>
@@ -18,5 +17,5 @@
     <parent link="base_footprint"/>
     <child link="base_link"/>
-    <origin xyz="0 0 ${(wheel_outer_radius+wheel_zoff)}" rpy="0 0 0"/>
+    <origin xyz="0 0 ${(wheel_radius+wheel_zoff)}" rpy="0 0 0"/>
   </joint>
   <!-- Robot Base -->
@@ -151,8 +150,8 @@
       <origin xyz="0 0 0.0155" rpy="0 0 0"/>
       <geometry>
-        <cylinder radius="${wheel_outer_radius}" length="${wheel_height}"/>
+        <sphere radius="${wheel_radius}"/>
       </geometry>
     </collision>
-    <xacro:cylinder_inertia mass="${wheel_mass}" length="${wheel_height}" radius="${wheel_outer_radius}">
+    <xacro:cylinder_inertia mass="${wheel_mass}" length="${wheel_height}" radius="${wheel_radius}">
       <origin xyz="0 0 0" rpy="0 0 0"/>
     </xacro:cylinder_inertia>
@@ -162,5 +161,4 @@
     <child link="left_wheel"/>
     <origin xyz="-0.028 0.055 -${wheel_zoff}" rpy="${pi/2} 0 ${pi}"/>
-    <!-- <limit upper="3.1415" lower="-3.1415" effort="30" velocity="5.0"/> -->
     <axis xyz="0 0 1"/>
   </joint>
@@ -175,8 +173,9 @@
       <origin xyz="0 0 -0.0065" rpy="0 0 0"/>
       <geometry>
-        <cylinder radius="${wheel_outer_radius}" length="${wheel_height}"/>
+        <sphere radius="${wheel_radius}"/>
+        <!-- <cylinder radius="${wheel_radius}" length="${wheel_height}"/> -->
       </geometry>
     </collision>
-    <xacro:cylinder_inertia mass="${wheel_mass}" length="${wheel_height}" radius="${wheel_outer_radius}">
+    <xacro:cylinder_inertia mass="${wheel_mass}" length="${wheel_height}" radius="${wheel_radius}">
       <origin xyz="0 0 0" rpy="0 0 0"/>
     </xacro:cylinder_inertia>
@@ -186,5 +185,4 @@
     <child link="right_wheel"/>
     <origin xyz="-0.028 -0.065 -${wheel_zoff}" rpy="${pi/2} 0 ${-pi}"/>
-    <!-- <limit upper="3.1415" lower="-3.1415" effort="30" velocity="5.0"/> -->
     <axis xyz="0 0 1"/>
   </joint>
