Commit message: Fixed xacro issue

File: models/lidarbot.urdf.xacro (robot description, xacro)
@@ -1,6 +1,6 @@
 <?xml version="1.0" ?>
 <robot name="lidarbot" xmlns:xacro="http://ros.org/wiki/xacro">
-    <xacro:include filename="lidarbot_core.xacro" />
-    <!-- <xacro:include filename="ros2_control.xacro"/> -->
+    <xacro:include filename="lidarbot_core.xacro"/>
+        <!-- <xacro:include filename="ros2_control.xacro"/> -->
     <xacro:include filename="camera.xacro"/>
     <xacro:include filename="imu.xacro"/>

File: models/lidarbot_core.xacro (robot description, xacro)
@@ -25,6 +25,6 @@
         <origin xyz="0 0 ${-wheel_zoff}" rpy="0 0 0"/>
           <geometry>
-              <mesh filename="package://real_lidarbot/models/lidarbot_description/meshes/robot_base_link.dae" />
-          </geometryk>
+              <mesh filename="package://real_lidarbot/models/lidarbot_description/meshes/robot_base.dae" />
+          </geometry>
       </visual>
       <collision>

Commit message: Spawn diff_controller and joint_state_broadcaster only if use_ros2_control is set to true

File: models/lidarbot.urdf.xacro (robot description, xacro)
@@ -3,15 +3,9 @@
     <xacro:arg name="use_ros2_control" default="true"/>
     <xacro:include filename="lidarbot_core.xacro"/>
-    <!-- <xacro:if value="$(arg use_ros2_control)">
+    <xacro:if value="$(arg use_ros2_control)">
         <xacro:include filename="ros2_control.xacro"/>
     </xacro:if>
     <xacro:unless value="$(arg use_ros2_control)">
         <xacro:include filename="gazebo_control.xacro"/>
-    </xacro:unless> -->
-    <xacro:if value="$(arg use_ros2_control)">
-        <xacro:include filename="ros2_control.xacro" />
-    </xacro:if>
-    <xacro:unless value="$(arg use_ros2_control)">
-        <xacro:include filename="gazebo_control.xacro" />
     </xacro:unless>
     <xacro:include filename="camera.xacro"/>

File: models/lidarbot_core.xacro (robot description, xacro)
@@ -174,5 +174,4 @@
       <geometry>
         <sphere radius="${wheel_radius}"/>
-        <!-- <cylinder radius="${wheel_radius}" length="${wheel_height}"/> -->
       </geometry>
     </collision>
