Commit message: Minor changes to ros2 control xacro

File: models/ros2_control.xacro (robot description, xacro)
@@ -2,28 +2,28 @@
 <robot xmlns:xacro="http://ros.org/wiki/xacro">
   <ros2_control name='GazeboSystem' type='system'>
-      <hardware>
-        <plugin>gazebo_ros2_control/GazeboSystem</plugin>
-      </hardware>
-      <joint name='left_wheel_joint'>
-        <command_interface name='velocity'>
-          <param name='min'>-10</param>
-          <param name='max'>10</param>
-        </command_interface>
-        <state_interface name='velocity'/>
-        <state_interface name='position'/>
-      </joint>
-      <joint name='right_wheel_joint'>
-        <command_interface name='velocity'>
-          <param name='min'>-10</param>
-          <param name='max'>10</param>
-        </command_interface>
-        <state_interface name='velocity'/>
-        <state_interface name='position'/>
-      </joint>
-    </ros2_control>
-    <gazebo>
-      <plugin name='lidarbot_ros2_control' filename='libgazebo_ros2_control.so'>
-        <parameters>$(find real_lidarbot)/config/my_controllers.yaml</parameters>
-      </plugin>
-    </gazebo>
+    <hardware>
+      <plugin>gazebo_ros2_control/GazeboSystem</plugin>
+    </hardware>
+    <joint name='left_wheel_joint'>
+      <command_interface name='velocity'>
+        <param name='min'>-10</param>
+        <param name='max'>10</param>
+      </command_interface>
+      <state_interface name='velocity'/>
+      <state_interface name='position'/>
+    </joint>
+    <joint name='right_wheel_joint'>
+      <command_interface name='velocity'>
+        <param name='min'>-10</param>
+        <param name='max'>10</param>
+      </command_interface>
+      <state_interface name='velocity'/>
+      <state_interface name='position'/>
+    </joint>
+  </ros2_control>
+  <gazebo>
+    <plugin name='gazebo_ros2_control' filename='libgazebo_ros2_control.so'>
+      <parameters>$(find real_lidarbot)/config/my_controllers.yaml</parameters>
+    </plugin>
+  </gazebo>
 </robot>

Commit message: Added files to test diff_drive_pca9685 functionality

File: models/ros2_control.xacro (robot description, xacro)
@@ -1,5 +1,30 @@
 <?xml version="1.0" ?>
 <robot xmlns:xacro="http://ros.org/wiki/xacro">
-  <ros2_control name='GazeboSystem' type='system'>
+  <ros2_control name='RealRobot' type='system'>
+    <hardware>
+      <plugin>diff_drive_pca9685/DiffDrivePCA9685</plugin>
+      <param name="right_wheel_name">left_wheel_joint</param>
+      <param name="left_wheel_name">right_wheel_joint</param>
+      <param name="loop_rate">30</param>
+      <param name="enc_ticks_per_rev">20</param>
+    </hardware>
+    <joint name='left_wheel_joint'>
+      <command_interface name='velocity'>
+        <param name='min'>-10</param>
+        <param name='max'>10</param>
+      </command_interface>
+      <state_interface name='velocity'/>
+      <state_interface name='position'/>
+    </joint>
+    <joint name='right_wheel_joint'>
+      <command_interface name='velocity'>
+        <param name='min'>-10</param>
+        <param name='max'>10</param>
+      </command_interface>
+      <state_interface name='velocity'/>
+      <state_interface name='position'/>
+    </joint>
+  </ros2_control>
+  <!-- <ros2_control name='GazeboSystem' type='system'>
     <hardware>
       <plugin>gazebo_ros2_control/GazeboSystem</plugin>
@@ -21,5 +46,5 @@
       <state_interface name='position'/>
     </joint>
-  </ros2_control>
+  </ros2_control> -->
   <gazebo>
     <plugin name='gazebo_ros2_control' filename='libgazebo_ros2_control.so'>
